File: KiCad/carrier/sheets/display_chain.kicad_sch (KiCad schematic)
At the start: 6 parts, among them U10 LT8618SX, U11 CBTL04GP054

Commit message: Rebuild all schematics with correct KiCad 10.0.2 format
Using exact format confirmed working with KiCad 10.0.2 on macOS.
All 16 schematics rebuilt:
- Shield root + 7 sub-sheets with hierarchical labels
- Carrier root + 7 sub-sheets with hierarchical labels

Format verified:
- version 20260101 (KiCad 10.0.2 SEXPR_SCHEMATIC_FILE_VERSION)
- generator_version 8.0
- Correct Sheetname/Sheetfile property names
- stroke/fill blocks on sheet definitions
- Proper hierarchical labels with effects blocks
Parts:
- removed C29: 100nF, Capacitor_SMD:C_0402_1005Metric, symbol Device:C
- removed C30: 10µF, Capacitor_SMD:C_0805_2012Metric, symbol Device:C
- removed J_DSI: MIPI DSI, Connector_FPC:Molex_503480-40_40pin_P0.5mm_Vertical, symbol Connector:FPC_40pin
- removed J_HDMI: Micro-HDMI, Connector_HDMI:Molex_47151-2001_Micro-HDMI_Horizontal, symbol Connector:Micro_HDMI
- removed U10: LT8618SX, Package_QFP:LQFP-56_10x10mm_P0.5mm, symbol Converter_DCDC:LT8618
- removed U11: CBTL04GP054, Package_DFN:DFN-16_3x3mm_P0.5mm, symbol Switch:CBTL04GP054
Changed lines of the file:
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@@
 (kicad_sch
-  (version 20260101)
-  (generator eeschema)
-  (generator_version "10.0.0")
-  (paper "A4")
-  (symbol (lib_id "Converter_DCDC:LT8618")
-    (at 30 30 0)
-    (unit 1)
-    (in_bom yes) (on_board yes)
-    (property "Reference" "U10"
-      (at 30 28.5 0)
-      (effects (font (size 1.27 1.27)))
-    )
-    (property "Value" "LT8618SX"
-      (at 30 31.5 0)
-      (effects (font (size 1.27 1.27)))
-    )
-    (property "Footprint" "Package_QFP:LQFP-56_10x10mm_P0.5mm"
-      (at 30 30 0)
-      (effects (font (size 1.27 1.27)) hide)
-    )
-    (instances
-      (project "uno_q_hub75_shield"
-        (path "/bc84562d-846a-4607-81a1-500b7991d137/f4a5b6c7-8d9e-0f1a-2b3c-4d5e6f7a8b9c"
-          (reference "U10") (unit 1)
-        )
-      )
-    )
-  )
-  (symbol (lib_id "Switch:CBTL04GP054")
-    (at 55 30 0)
-    (unit 1)
-    (in_bom yes) (on_board yes)
-    (property "Reference" "U11"
-      (at 55 28.5 0)
-      (effects (font (size 1.27 1.27)))
-    )
-    (property "Value" "CBTL04GP054"
-      (at 55 31.5 0)
-      (effects (font (size 1.27 1.27)))
-    )
-    (property "Footprint" "Package_DFN:DFN-16_3x3mm_P0.5mm"
-      (at 55 30 0)
-      (effects (font (size 1.27 1.27)) hide)
-    )
-    (instances
-      (project "uno_q_hub75_shield"
-        (path "/bc84562d-846a-4607-81a1-500b7991d137/f4a5b6c7-8d9e-0f1a-2b3c-4d5e6f7a8b9c"
-          (reference "U11") (unit 1)
-        )
-      )
-    )
-  )
-  (symbol (lib_id "Device:C")
-    (at 20 25 0)
-    (unit 1)
-    (in_bom yes) (on_board yes)
-    (property "Reference" "C29"
-      (at 20 23.5 0)
-      (effects (font (size 1.27 1.27)))
-    )
-    (property "Value" "100nF"
-      (at 20 26.5 0)
-      (effects (font (size 1.27 1.27)))
-    )
-    (property "Footprint" "Capacitor_SMD:C_0402_1005Metric"
-      (at 20 25 0)
-      (effects (font (size 1.27 1.27)) hide)
-    )
-    (instances
-      (project "uno_q_hub75_shield"
-        (path "/bc84562d-846a-4607-81a1-500b7991d137/f4a5b6c7-8d9e-0f1a-2b3c-4d5e6f7a8b9c"
-          (reference "C29") (unit 1)
-        )
-      )
-    )
-  )
-  (symbol (lib_id "Device:C")
-    (at 25 25 0)
-    (unit 1)
-    (in_bom yes) (on_board yes)
-    (property "Reference" "C30"
-      (at 25 23.5 0)
-      (effects (font (size 1.27 1.27)))
-    )
-    (property "Value" "10µF"
-      (at 25 26.5 0)
-      (effects (font (size 1.27 1.27)))
-    )
-    (property "Footprint" "Capacitor_SMD:C_0805_2012Metric"
-      (at 25 25 0)
-      (effects (font (size 1.27 1.27)) hide)
-    )
-    (instances
-      (project "uno_q_hub75_shield"
-        (path "/bc84562d-846a-4607-81a1-500b7991d137/f4a5b6c7-8d9e-0f1a-2b3c-4d5e6f7a8b9c"
-          (reference "C30") (unit 1)
-        )
-      )
-    )
-  )
-  (symbol (lib_id "Connector:Micro_HDMI")
-    (at 75 30 0)
-    (unit 1)
-    (in_bom yes) (on_board yes)
-    (property "Reference" "J_HDMI"
-      (at 75 28.5 0)
-      (effects (font (size 1.27 1.27)))
-    )
-    (property "Value" "Micro-HDMI"
-      (at 75 31.5 0)
-      (effects (font (size 1.27 1.27)))
-    )
-    (property "Footprint" "Connector_HDMI:Molex_47151-2001_Micro-HDMI_Horizontal"
-      (at 75 30 0)
-      (effects (font (size 1.27 1.27)) hide)
-    )
-    (instances
-      (project "uno_q_hub75_shield"
-        (path "/bc84562d-846a-4607-81a1-500b7991d137/f4a5b6c7-8d9e-0f1a-2b3c-4d5e6f7a8b9c"
-          (reference "J_HDMI") (unit 1)
-        )
-      )
-    )
-  )
-  (symbol (lib_id "Connector:FPC_40pin")
-    (at 75 40 0)
-    (unit 1)
-    (in_bom yes) (on_board yes)
-    (property "Reference" "J_DSI"
-      (at 75 38.5 0)
-      (effects (font (size 1.27 1.27)))
-    )
-    (property "Value" "MIPI DSI"
-      (at 75 41.5 0)
-      (effects (font (size 1.27 1.27)))
-    )
-    (property "Footprint" "Connector_FPC:Molex_503480-40_40pin_P0.5mm_Vertical"
-      (at 75 40 0)
-      (effects (font (size 1.27 1.27)) hide)
-    )
-    (instances
-      (project "uno_q_hub75_shield"
-        (path "/bc84562d-846a-4607-81a1-500b7991d137/f4a5b6c7-8d9e-0f1a-2b3c-4d5e6f7a8b9c"
-          (reference "J_DSI") (unit 1)
-        )
-      )
-    )
-  )
-  (hierarchical_label "+5V"
-    (shape input)
-    (at 10 20 0)
-    (effects (font (size 1.27 1.27)) (justify left))
-  )
-  (hierarchical_label "+3V3"
-    (shape input)
-    (at 10 25 0)
-    (effects (font (size 1.27 1.27)) (justify left))
-  )
-  (hierarchical_label "DGND"
-    (shape input)
-    (at 10 30 0)
-    (effects (font (size 1.27 1.27)) (justify left))
-  )
-  (sheet_instances
-    (path "/"
-      (page "1")
-    )
-  )
+	(version 20260101)
+	(generator "eeschema")
+	(generator_version "8.0")
+	(paper "A4")
+	(hierarchical_label "+3V3"
+		(shape input)
+		(at 10 25 0)
+		(fields_autoplaced yes)
+		(effects
+			(font
+				(size 1.27 1.27)
+			)
+			(justify left)
+		)
+		(uuid "f4a5b6c7-8d9e-0f1a-2b3c-4d5e6f7a8b9c-hl00")
+	)
+	(hierarchical_label "DGND"
+		(shape input)
+		(at 10 30 0)
+		(fields_autoplaced yes)
+		(effects
+			(font
+				(size 1.27 1.27)
+			)
+			(justify left)
+		)
+		(uuid "f4a5b6c7-8d9e-0f1a-2b3c-4d5e6f7a8b9c-hl01")
+	)
+	(hierarchical_label "MIPI_CLK"
+		(shape input)
+		(at 85 25 0)
+		(fields_autoplaced yes)
+		(effects
+			(font
+				(size 1.27 1.27)
+			)
+			(justify left)
+		)
+		(uuid "f4a5b6c7-8d9e-0f1a-2b3c-4d5e6f7a8b9c-hl02")
+	)
+	(hierarchical_label "MIPI_DATA"
+		(shape input)
+		(at 85 30 0)
+		(fields_autoplaced yes)
+		(effects
+			(font
+				(size 1.27 1.27)
+			)
+			(justify left)
+		)
+		(uuid "f4a5b6c7-8d9e-0f1a-2b3c-4d5e6f7a8b9c-hl03")
+	)
+	(sheet_instances
+		(path "/"
+			(page "5")
+		)
+	)
 )
