File: KiCad/carrier/sheets/esp32c6_radio.kicad_sch (KiCad schematic)
At the start: 11 parts, among them U6 ESP32-C6-MINI-1

Commit message: Rebuild all schematics as valid KiCad 10 format (version 20260326)
Complete rewrite from scratch using Python generator (kicad10_gen.py).
All 16 files verified parseable with kicad-skip and structurally
compliant with the KiCad schematic file format specification.

Format compliance per dev-docs.kicad.org/en/file-formats/sexpr-schematic/:
  - version 20260326 (KiCad 10 SEXPR_SCHEMATIC_FILE_VERSION)
  - generator_version 10.0.0
  - Root (uuid) in every schematic file header
  - Every symbol instance has: (uuid UUID) + (instances (project NAME (path /ROOT/SHEET (reference REF)(unit N))))
  - Every hierarchical_label has: (uuid UUID)
  - Every sheet block has: (uuid UUID) + (instances (project NAME (path /ROOT_UUID (page N))))
  - Every sheet pin has: (uuid UUID)
  - Every text element has: (uuid UUID)
  - Root schematics have: (sheet_instances (path '/' (page '1')))
  - lib_symbols: pin type uses 'TYPE line' format (e.g. 'input line')
  - All property effects use correct KiCad 10 token syntax
  - Stable UUIDs via seed files (shield_uuids.json, carrier_uuids.json)

Shield (8 files, stable root UUID: bc84562d-846a-4607-81a1-500b7991d137):
  uno_q_hub75_shield.kicad_sch      root, 7 hierarchical sheets
  sheets/power.kicad_sch            AMS1117-3.3 LDO, FB1, indicators (17 syms)
  sheets/esp32s3.kicad_sch          ESP32-S3-WROOM-1-N16R8, USB-C (9 syms)
  sheets/hub75_driver.kicad_sch     SN74HCT245PW x2, HUB75 IDC (10 syms)
  sheets/audio_codec.kicad_sch      ES8388, DC-block caps, J_OUT/J_MIC (19 syms)
  sheets/display.kicad_sch          FPC_22pin, GT911 pullups, JP1 (7 syms)
  sheets/uno_q_interface.kicad_sch  J2 SPI3, J3 UART debug (2 syms)
  sheets/connectivity.kicad_sch     Qwiic x2, Grove x5 (10 syms)

Carrier (8 files, stable root UUID: a7d62ed3-8e95-4e64-b6df-722c91664a1a):
  uno_q_super_carrier.kicad_sch     root, 10 hierarchical sheets
  sheets/power.kicad_sch            TPS54331DR buck, AMS1117, dual VIN/HUB75 (33 syms)
  sheets/uno_q_mounting.kicad_sch   B1 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
Parts:
- removed C_C1: 100nF 10V X7R 0402, Capacitor_SMD:C_0402_1005Metric, symbol C
- removed C_C2: 10µF 10V X5R 0805, Capacitor_SMD:C_0805_2012Metric, symbol C
- removed J_ANT: U.FL_Ext_2.4GHz, symbol U_FL_CONN
- removed J_C6_USB: C6_DEBUG_USB, symbol USB_C_RECEPTACLE
- removed R_ANT_EXT: 0Ω EXT_ANT DNP, symbol R
- removed R_ANT_PCB: 0Ω PCB_ANT (default), symbol R
- removed R_C1, R_C2: 10kΩ 1% 0402, symbol R
- removed R_C3, R_C4: 5.1kΩ 1% 0402, symbol R
- removed U6: ESP32-C6-MINI-1, symbol ESP32-C6-MINI-1
- added C_C1: 100nF 10V X7R 0402, Capacitor_SMD:C_0402_1005Metric, symbol Device:C
- added C_C2: 10µF 10V X5R 0805, Capacitor_SMD:C_0805_2012Metric, symbol Device:C
- added J_ANT: U.FL_Ext_2.4GHz, Connector_Coaxial:U.FL_Hirose_U.FL-R-SMT-1_Vertical, symbol HybotixParts:UFL_Connector
- added J_C6_USB: C6_DEBUG_USB, Connector_USB:USB_C_Receptacle_GCT_USB4135_FlipMounted, symbol HybotixParts:USB_C
- added R_ANT_EXT: 0Ω EXT_ANT_DNP, Resistor_SMD:R_0402_1005Metric, symbol Device:R
- added R_ANT_PCB: 0Ω PCB_ANT_default, Resistor_SMD:R_0402_1005Metric, symbol Device:R
- added R_C1: 10kΩ 1% 0402 EN pullup, Resistor_SMD:R_0402_1005Metric, symbol Device:R
- added R_C2: 10kΩ 1% 0402 GPIO0 pullup, Resistor_SMD:R_0402_1005Metric, symbol Device:R
- added R_C3: 5.1kΩ 1% 0402 CC1, Resistor_SMD:R_0402_1005Metric, symbol Device:R
- added R_C4: 5.1kΩ 1% 0402 CC2, Resistor_SMD:R_0402_1005Metric, symbol Device:R
- added U6: ESP32-C6-MINI-1, RF_Module:ESP32-C6-MINI-1, symbol HybotixParts:ESP32-C6-MINI-1
Other:
- note added: "ESP32-C6 ANTENNA SELECTION:\nR_ANT_PCB (0Ω populated): RF → MINI-1 PCB trace antenna\nR_ANT_EXT (0Ω DNP): RF → J_ANT U.FL external antenna\nNEVER populate both resistors simultaneously\nFor external antenna: swap to MINI-1U + populate R_ANT_EXT only\nAntenna keepout: 3mm clear of all copper all layers\nModule PCB edge placement: antenna must overhang carrier board\n50Ω RF trace: outer layer only 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"
- note removed: "ESP32-C6 RADIO CO-PROCESSOR NOTES: ANTENNA SELECTION (Espressif HW Design Guidelines §RF): R_ANT_PCB (0Ω, populated): routes C6 RF pad to MINI-1 PCB trace antenna R_ANT_EXT (0Ω, DNP): routes C6 RF pad to J_ANT U.FL connector Only ONE resistor may be populated. Never both simultaneously. PCB RF trace: 50Ω impedance controlled, outer layer only, no vias, 135° bends Keepout under J_ANT U.FL: all lay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"

Commit message: REBUILD: Minimal KiCad 10.0.2 compatible schematic files
Completely rebuilt all 16 schematic files using absolute minimum structure
that KiCad 10.0.2 on macOS will accept:

Root schematics (2 files):
- uno_q_hub75_shield.kicad_sch (7 sheets)
- uno_q_super_carrier.kicad_sch (7 sheets)

Sub-sheets (14 files):
- All 7 shield sub-sheets
- All 7 carrier sub-sheets

Format: Minimal valid structure — only mandatory elements
- (kicad_sch version 20260326)
- (generator eeschema, generator_version 10.0.0)
- (uuid) for each file
- (lib_symbols) empty section
- (sheet) blocks with uuid + instances
- (sheet_instances) at end
- Hierarchical labels with uuid

No complex symbol instances, no wires, no graphic elements —
just the bare structure KiCad needs to load the files.
Parts:
- removed C_C1: 100nF 10V X7R 0402, Capacitor_SMD:C_0402_1005Metric, symbol Device:C
- removed C_C2: 10µF 10V X5R 0805, Capacitor_SMD:C_0805_2012Metric, symbol Device:C
- removed J_ANT: U.FL_Ext_2.4GHz, Connector_Coaxial:U.FL_Hirose_U.FL-R-SMT-1_Vertical, symbol HybotixParts:UFL_Connector
- removed J_C6_USB: C6_DEBUG_USB, Connector_USB:USB_C_Receptacle_GCT_USB4135_FlipMounted, symbol HybotixParts:USB_C
- removed R_ANT_EXT: 0Ω EXT_ANT_DNP, Resistor_SMD:R_0402_1005Metric, symbol Device:R
- removed R_ANT_PCB: 0Ω PCB_ANT_default, Resistor_SMD:R_0402_1005Metric, symbol Device:R
- removed R_C1: 10kΩ 1% 0402 EN pullup, Resistor_SMD:R_0402_1005Metric, symbol Device:R
- removed R_C2: 10kΩ 1% 0402 GPIO0 pullup, Resistor_SMD:R_0402_1005Metric, symbol Device:R
- removed R_C3: 5.1kΩ 1% 0402 CC1, Resistor_SMD:R_0402_1005Metric, symbol Device:R
- removed R_C4: 5.1kΩ 1% 0402 CC2, Resistor_SMD:R_0402_1005Metric, symbol Device:R
- removed U6: ESP32-C6-MINI-1, RF_Module:ESP32-C6-MINI-1, symbol HybotixParts:ESP32-C6-MINI-1
Other:
- note removed: "ESP32-C6 ANTENNA SELECTION:\nR_ANT_PCB (0Ω populated): RF → MINI-1 PCB trace antenna\nR_ANT_EXT (0Ω DNP): RF → J_ANT U.FL external antenna\nNEVER populate both resistors simultaneously\nFor external antenna: swap to MINI-1U + populate R_ANT_EXT only\nAntenna keepout: 3mm clear of all copper all layers\nModule PCB edge placement: antenna must overhang carrier board\n50Ω RF trace: outer layer only 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"
- company: Hybrid RobotiX -> (none)
- title: UNO Q Super Carrier — ESP32-C6 Radio Co-Processor -> (none)
