File: KiCad/carrier/sheets/esp32c6_radio.kicad_sch (KiCad schematic)
At the start: 0 parts

Commit message: Add carrier schematic generator + rebuild all carrier schematics with complete BOM
Generator:
- build_carrier_complete.py: Carrier-specific generator with all 7 sheets + root

Carrier rebuilt with complete component list from BOM:
- power.kicad_sch: TPS54331 buck, dual VIN support, feedback divider (13 components)
- uno_q_mounting.kicad_sch: Samtec FTSH-130-01 mezzanine connectors (2 components + power/signals)
- esp32c6_radio.kicad_sch: ESP32-C6-MINI-1 module, antenna selection, U.FL connector (6 components)
- display_chain.kicad_sch: LT8618SX MIPI→HDMI, CBTL04GP054 switch, Micro-HDMI (5 components)
- rpi5_interface.kicad_sch: 40-pin GPIO, 24C32 HAT EEPROM, CSI0/CSI1 FPC (8 components)
- level_shift.kicad_sch: TXS0108E x2 level shifters for MPU GPIO (2 components)
- expansion.kicad_sch: Qwiic x2, Grove x5 with pullups (7 components)
- uno_q_super_carrier.kicad_sch: Root schematic with all 7 sheets

All 8 files verified with kicad-skip parser (KiCad 10.0.2 compatible).
Regenerable from scripts - ready to open in KiCad 10.0.2.
Parts:
- added C27: 100nF, Capacitor_SMD:C_0402_1005Metric, symbol Device:C
- added C28: 10µF, Capacitor_SMD:C_0805_2012Metric, symbol Device:C
- added J_ANT: U.FL, Connector_Coaxial:HIROSE_UFL_2013_E, symbol HybotixParts:UFL_Connector
- added J_C6_USB: C6 USB, Connector_USB:USB_C_Receptacle_GCT_USB4135-GF-A_Horizontal, symbol HybotixParts:USB_C_Receptacle
- added R_ANT_EXT: DNP, Resistor_SMD:R_0402_1005Metric, symbol Device:R
- added R_ANT_PCB: 0Ω, Resistor_SMD:R_0402_1005Metric, symbol Device:R
- added U9: ESP32-C6-MINI-1, Package_BGA:ESP32-C6-MINI-1_18x18.5mm_P0.4mm, symbol HybotixParts:ESP32-C6-MINI-1
Changed lines of the file:
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@@
   (generator_version "10.0.0")
   (paper "A4")
+  (symbol (lib_id "HybotixParts:ESP32-C6-MINI-1")
+    (at 30 30 0)
+    (unit 1)
+    (in_bom yes) (on_board yes)
+    (property "Reference" "U9"
+      (at 30 28.5 0)
+      (effects (font (size 1.27 1.27)))
+    )
+    (property "Value" "ESP32-C6-MINI-1"
+      (at 30 31.5 0)
+      (effects (font (size 1.27 1.27)))
+    )
+    (property "Footprint" "Package_BGA:ESP32-C6-MINI-1_18x18.5mm_P0.4mm"
+      (at 30 30 0)
+      (effects (font (size 1.27 1.27)) hide)
+    )
+    (instances
+      (project "uno_q_hub75_shield"
+        (path "/bc84562d-846a-4607-81a1-500b7991d137/SHEETUUID"
+          (reference "U9") (unit 1)
+        )
+      )
+    )
+  )
+  (symbol (lib_id "Device:C")
+    (at 20 30 0)
+    (unit 1)
+    (in_bom yes) (on_board yes)
+    (property "Reference" "C27"
+      (at 20 28.5 0)
+      (effects (font (size 1.27 1.27)))
+    )
+    (property "Value" "100nF"
+      (at 20 31.5 0)
+      (effects (font (size 1.27 1.27)))
+    )
+    (property "Footprint" "Capacitor_SMD:C_0402_1005Metric"
+      (at 20 30 0)
+      (effects (font (size 1.27 1.27)) hide)
+    )
+    (instances
+      (project "uno_q_hub75_shield"
+        (path "/bc84562d-846a-4607-81a1-500b7991d137/SHEETUUID"
+          (reference "C27") (unit 1)
+        )
+      )
+    )
+  )
+  (symbol (lib_id "Device:C")
+    (at 25 30 0)
+    (unit 1)
+    (in_bom yes) (on_board yes)
+    (property "Reference" "C28"
+      (at 25 28.5 0)
+      (effects (font (size 1.27 1.27)))
+    )
+    (property "Value" "10µF"
+      (at 25 31.5 0)
+      (effects (font (size 1.27 1.27)))
+    )
+    (property "Footprint" "Capacitor_SMD:C_0805_2012Metric"
+      (at 25 30 0)
+      (effects (font (size 1.27 1.27)) hide)
+    )
+    (instances
+      (project "uno_q_hub75_shield"
+        (path "/bc84562d-846a-4607-81a1-500b7991d137/SHEETUUID"
+          (reference "C28") (unit 1)
+        )
+      )
+    )
+  )
+  (symbol (lib_id "Device:R")
+    (at 50 25 0)
+    (unit 1)
+    (in_bom yes) (on_board yes)
+    (property "Reference" "R_ANT_PCB"
+      (at 50 23.5 0)
+      (effects (font (size 1.27 1.27)))
+    )
+    (property "Value" "0Ω"
+      (at 50 26.5 0)
+      (effects (font (size 1.27 1.27)))
+    )
+    (property "Footprint" "Resistor_SMD:R_0402_1005Metric"
+      (at 50 25 0)
+      (effects (font (size 1.27 1.27)) hide)
+    )
+    (instances
+      (project "uno_q_hub75_shield"
+        (path "/bc84562d-846a-4607-81a1-500b7991d137/SHEETUUID"
+          (reference "R_ANT_PCB") (unit 1)
+        )
+      )
+    )
+  )
+  (symbol (lib_id "Device:R")
+    (at 55 25 0)
+    (unit 1)
+    (in_bom yes) (on_board yes)
+    (property "Reference" "R_ANT_EXT"
+      (at 55 23.5 0)
+      (effects (font (size 1.27 1.27)))
+    )
+    (property "Value" "DNP"
+      (at 55 26.5 0)
+      (effects (font (size 1.27 1.27)))
+    )
+    (property "Footprint" "Resistor_SMD:R_0402_1005Metric"
+      (at 55 25 0)
+      (effects (font (size 1.27 1.27)) hide)
+    )
+    (instances
+      (project "uno_q_hub75_shield"
+        (path "/bc84562d-846a-4607-81a1-500b7991d137/SHEETUUID"
+          (reference "R_ANT_EXT") (unit 1)
+        )
+      )
+    )
+  )
+  (symbol (lib_id "HybotixParts:UFL_Connector")
+    (at 60 30 0)
+    (unit 1)
+    (in_bom yes) (on_board yes)
+    (property "Reference" "J_ANT"
+      (at 60 28.5 0)
+      (effects (font (size 1.27 1.27)))
+    )
+    (property "Value" "U.FL"
+      (at 60 31.5 0)
+      (effects (font (size 1.27 1.27)))
+    )
+    (property "Footprint" "Connector_Coaxial:HIROSE_UFL_2013_E"
+      (at 60 30 0)
+      (effects (font (size 1.27 1.27)) hide)
+    )
+    (instances
+      (project "uno_q_hub75_shield"
+        (path "/bc84562d-846a-4607-81a1-500b7991d137/SHEETUUID"
+          (reference "J_ANT") (unit 1)
+        )
+      )
+    )
+  )
+  (symbol (lib_id "HybotixParts:USB_C_Receptacle")
+    (at 70 30 0)
+    (unit 1)
+    (in_bom yes) (on_board yes)
+    (property "Reference" "J_C6_USB"
+      (at 70 28.5 0)
+      (effects (font (size 1.27 1.27)))
+    )
+    (property "Value" "C6 USB"
+      (at 70 31.5 0)
+      (effects (font (size 1.27 1.27)))
+    )
+    (property "Footprint" "Connector_USB:USB_C_Receptacle_GCT_USB4135-GF-A_Horizontal"
+      (at 70 30 0)
+      (effects (font (size 1.27 1.27)) hide)
+    )
+    (instances
+      (project "uno_q_hub75_shield"
+        (path "/bc84562d-846a-4607-81a1-500b7991d137/SHEETUUID"
+          (reference "J_C6_USB") (unit 1)
+        )
+      )
+    )
+  )
   (hierarchical_label "+3V3"
     (shape input)
-    (at 10 10 0)
+    (at 10 25 0)
     (effects (font (size 1.27 1.27)) (justify left))
   )
+  (hierarchical_label "DGND"
+    (shape input)
+    (at 10 35 0)
+    (effects (font (size 1.27 1.27)) (justify left))
+  )
+  (hierarchical_label "S3_C6_TX"
+    (shape input)
+    (at 10 40 0)
+    (effects (font (size 1.27 1.27)) (justify left))
+  )
+  (hierarchical_label "S3_C6_RX"
+    (shape output)
+    (at 10 45 0)
+    (effects (font (size 1.27 1.27)) (justify left))
+  )
