File: KiCad/carrier/sheets/expansion.kicad_sch (KiCad schematic)
At the start: 9 parts, among them J15 Qwiic, J16 Qwiic, J17 Grove PSSI, J18 Grove I2C4, J19 Grove, J20 Grove, J21 Grove OpAmp

Commit message: Rebuild all schematics with correct KiCad 10.0.2 format
Using exact format confirmed working with KiCad 10.0.2 on macOS.
All 16 schematics rebuilt:
- Shield root + 7 sub-sheets with hierarchical labels
- Carrier root + 7 sub-sheets with hierarchical labels

Format verified:
- version 20260101 (KiCad 10.0.2 SEXPR_SCHEMATIC_FILE_VERSION)
- generator_version 8.0
- Correct Sheetname/Sheetfile property names
- stroke/fill blocks on sheet definitions
- Proper hierarchical labels with effects blocks
Parts:
- removed J15, J16: Qwiic, Connector_JST:JST_SH_BM04B-SRSS-TB_1x04-1MP_P1.0mm_Vertical, symbol Connector:Conn_01x04_Pin
- removed J17: Grove PSSI, Connector_Grove:Grove_4pin_Vertical, symbol Connector:Conn_01x04_Pin
- removed J18: Grove I2C4, Connector_Grove:Grove_4pin_Vertical, symbol Connector:Conn_01x04_Pin
- removed J19, J20: Grove, Connector_Grove:Grove_4pin_Vertical, symbol Connector:Conn_01x04_Pin
- removed J21: Grove OpAmp, Connector_Grove:Grove_4pin_Vertical, symbol Connector:Conn_01x04_Pin
- removed R24, R25: 4.7kΩ, Resistor_SMD:R_0402_1005Metric, symbol Device:R
