File: KiCad/carrier/sheets/level_shift.kicad_sch (KiCad schematic)
At the start: 4 parts

Commit message: Rebuild all schematics with correct KiCad 10.0.2 format
Using exact format confirmed working with KiCad 10.0.2 on macOS.
All 16 schematics rebuilt:
- Shield root + 7 sub-sheets with hierarchical labels
- Carrier root + 7 sub-sheets with hierarchical labels

Format verified:
- version 20260101 (KiCad 10.0.2 SEXPR_SCHEMATIC_FILE_VERSION)
- generator_version 8.0
- Correct Sheetname/Sheetfile property names
- stroke/fill blocks on sheet definitions
- Proper hierarchical labels with effects blocks
Parts:
- removed C32, C33: 100nF, Capacitor_SMD:C_0402_1005Metric, symbol Device:C
- removed U_LS1, U_LS2: TXS0108E, Package_SO:TSSOP-20_4.4x6.5mm_P0.65mm, symbol Converter_Level:TXS0108E
Changed lines of the file:
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@@
 (kicad_sch
-  (version 20260101)
-  (generator eeschema)
-  (generator_version "10.0.0")
-  (paper "A4")
-  (symbol (lib_id "Converter_Level:TXS0108E")
-    (at 30 25 0)
-    (unit 1)
-    (in_bom yes) (on_board yes)
-    (property "Reference" "U_LS1"
-      (at 30 23.5 0)
-      (effects (font (size 1.27 1.27)))
-    )
-    (property "Value" "TXS0108E"
-      (at 30 26.5 0)
-      (effects (font (size 1.27 1.27)))
-    )
-    (property "Footprint" "Package_SO:TSSOP-20_4.4x6.5mm_P0.65mm"
-      (at 30 25 0)
-      (effects (font (size 1.27 1.27)) hide)
-    )
-    (instances
-      (project "uno_q_hub75_shield"
-        (path "/bc84562d-846a-4607-81a1-500b7991d137/b6c7d8e9-0f1a-2b3c-4d5e-6f7a8b9c0d1e"
-          (reference "U_LS1") (unit 1)
-        )
-      )
-    )
-  )
-  (symbol (lib_id "Converter_Level:TXS0108E")
-    (at 50 25 0)
-    (unit 1)
-    (in_bom yes) (on_board yes)
-    (property "Reference" "U_LS2"
-      (at 50 23.5 0)
-      (effects (font (size 1.27 1.27)))
-    )
-    (property "Value" "TXS0108E"
-      (at 50 26.5 0)
-      (effects (font (size 1.27 1.27)))
-    )
-    (property "Footprint" "Package_SO:TSSOP-20_4.4x6.5mm_P0.65mm"
-      (at 50 25 0)
-      (effects (font (size 1.27 1.27)) hide)
-    )
-    (instances
-      (project "uno_q_hub75_shield"
-        (path "/bc84562d-846a-4607-81a1-500b7991d137/b6c7d8e9-0f1a-2b3c-4d5e-6f7a8b9c0d1e"
-          (reference "U_LS2") (unit 1)
-        )
-      )
-    )
-  )
-  (symbol (lib_id "Device:C")
-    (at 20 25 0)
-    (unit 1)
-    (in_bom yes) (on_board yes)
-    (property "Reference" "C32"
-      (at 20 23.5 0)
-      (effects (font (size 1.27 1.27)))
-    )
-    (property "Value" "100nF"
-      (at 20 26.5 0)
-      (effects (font (size 1.27 1.27)))
-    )
-    (property "Footprint" "Capacitor_SMD:C_0402_1005Metric"
-      (at 20 25 0)
-      (effects (font (size 1.27 1.27)) hide)
-    )
-    (instances
-      (project "uno_q_hub75_shield"
-        (path "/bc84562d-846a-4607-81a1-500b7991d137/b6c7d8e9-0f1a-2b3c-4d5e-6f7a8b9c0d1e"
-          (reference "C32") (unit 1)
-        )
-      )
-    )
-  )
-  (symbol (lib_id "Device:C")
-    (at 40 25 0)
-    (unit 1)
-    (in_bom yes) (on_board yes)
-    (property "Reference" "C33"
-      (at 40 23.5 0)
-      (effects (font (size 1.27 1.27)))
-    )
-    (property "Value" "100nF"
-      (at 40 26.5 0)
-      (effects (font (size 1.27 1.27)))
-    )
-    (property "Footprint" "Capacitor_SMD:C_0402_1005Metric"
-      (at 40 25 0)
-      (effects (font (size 1.27 1.27)) hide)
-    )
-    (instances
-      (project "uno_q_hub75_shield"
-        (path "/bc84562d-846a-4607-81a1-500b7991d137/b6c7d8e9-0f1a-2b3c-4d5e-6f7a8b9c0d1e"
-          (reference "C33") (unit 1)
-        )
-      )
-    )
-  )
-  (hierarchical_label "VIN_1V8_REF"
-    (shape input)
-    (at 10 20 0)
-    (effects (font (size 1.27 1.27)) (justify left))
-  )
-  (hierarchical_label "+3V3"
-    (shape input)
-    (at 10 30 0)
-    (effects (font (size 1.27 1.27)) (justify left))
-  )
-  (hierarchical_label "DGND"
-    (shape input)
-    (at 10 35 0)
-    (effects (font (size 1.27 1.27)) (justify left))
-  )
-  (sheet_instances
-    (path "/"
-      (page "1")
-    )
-  )
+	(version 20260101)
+	(generator "eeschema")
+	(generator_version "8.0")
+	(paper "A4")
+	(hierarchical_label "+3V3"
+		(shape input)
+		(at 10 25 0)
+		(fields_autoplaced yes)
+		(effects
+			(font
+				(size 1.27 1.27)
+			)
+			(justify left)
+		)
+		(uuid "b6c7d8e9-0f1a-2b3c-4d5e-6f7a8b9c0d1e-hl00")
+	)
+	(hierarchical_label "DGND"
+		(shape input)
+		(at 10 30 0)
+		(fields_autoplaced yes)
+		(effects
+			(font
+				(size 1.27 1.27)
+			)
+			(justify left)
+		)
+		(uuid "b6c7d8e9-0f1a-2b3c-4d5e-6f7a8b9c0d1e-hl01")
+	)
+	(sheet_instances
+		(path "/"
+			(page "7")
+		)
+	)
 )
