File: KiCad/carrier/sheets/rpi5_interface.kicad_sch (KiCad schematic)
At the start: 7 parts

Commit message: Rebuild all schematics as valid KiCad 10 format (version 20260326)
Complete rewrite from scratch using Python generator (kicad10_gen.py).
All 16 files verified parseable with kicad-skip and structurally
compliant with the KiCad schematic file format specification.

Format compliance per dev-docs.kicad.org/en/file-formats/sexpr-schematic/:
  - version 20260326 (KiCad 10 SEXPR_SCHEMATIC_FILE_VERSION)
  - generator_version 10.0.0
  - Root (uuid) in every schematic file header
  - Every symbol instance has: (uuid UUID) + (instances (project NAME (path /ROOT/SHEET (reference REF)(unit N))))
  - Every hierarchical_label has: (uuid UUID)
  - Every sheet block has: (uuid UUID) + (instances (project NAME (path /ROOT_UUID (page N))))
  - Every sheet pin has: (uuid UUID)
  - Every text element has: (uuid UUID)
  - Root schematics have: (sheet_instances (path '/' (page '1')))
  - lib_symbols: pin type uses 'TYPE line' format (e.g. 'input line')
  - All property effects use correct KiCad 10 token syntax
  - Stable UUIDs via seed files (shield_uuids.json, carrier_uuids.json)

Shield (8 files, stable root UUID: bc84562d-846a-4607-81a1-500b7991d137):
  uno_q_hub75_shield.kicad_sch      root, 7 hierarchical sheets
  sheets/power.kicad_sch            AMS1117-3.3 LDO, FB1, indicators (17 syms)
  sheets/esp32s3.kicad_sch          ESP32-S3-WROOM-1-N16R8, USB-C (9 syms)
  sheets/hub75_driver.kicad_sch     SN74HCT245PW x2, HUB75 IDC (10 syms)
  sheets/audio_codec.kicad_sch      ES8388, DC-block caps, J_OUT/J_MIC (19 syms)
  sheets/display.kicad_sch          FPC_22pin, GT911 pullups, JP1 (7 syms)
  sheets/uno_q_interface.kicad_sch  J2 SPI3, J3 UART debug (2 syms)
  sheets/connectivity.kicad_sch     Qwiic x2, Grove x5 (10 syms)

Carrier (8 files, stable root UUID: a7d62ed3-8e95-4e64-b6df-722c91664a1a):
  uno_q_super_carrier.kicad_sch     root, 10 hierarchical sheets
  sheets/power.kicad_sch            TPS54331DR buck, AMS1117, dual VIN/HUB75 (33 syms)
  sheets/uno_q_mounting.kicad_sch   B1 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
Parts:
- removed J_CSI0: CSI0_RPi5_22pin, symbol FPC_22PIN_CSI
- removed J_CSI1: CSI1_RPi5_22pin, symbol FPC_22PIN_CSI
- removed J_GPIO40: RPi5_40PIN, symbol CONN_2x20_GPIO
- removed R_E1: 0Ω DNP (addr=0x50), symbol R
- removed R_E2, R_E3: 4.7kΩ 1% 0402, symbol R
- removed U_EEPROM: 24C32_HAT_ID, symbol EEPROM_24C32
- added J_CSI0: CSI0_RPi5_22pin, Connector_FFC-FPC:Molex_503480-2200_1x22-1MP_P0.50mm_Horizontal, symbol HybotixParts:FPC_22pin_0.5mm
- added J_CSI1: CSI1_RPi5_22pin, Connector_FFC-FPC:Molex_503480-2200_1x22-1MP_P0.50mm_Horizontal, symbol HybotixParts:FPC_22pin_0.5mm
- added J_GPIO40: RPi5_40PIN, Connector_PinHeader_2.54mm:PinHeader_2x20_P2.54mm_Vertical, symbol HybotixParts:GPIO40_RPi5
- added R_E1: 0Ω DNP A0=A1=A2=GND addr=0x50, Resistor_SMD:R_0402_1005Metric, symbol Device:R
- added R_E2: 4.7kΩ 1% 0402 ID_SD pullup, Resistor_SMD:R_0402_1005Metric, symbol Device:R
- added R_E3: 4.7kΩ 1% 0402 ID_SC pullup, Resistor_SMD:R_0402_1005Metric, symbol Device:R
- added U_EEPROM: 24C32_HAT_ID, Package_SO:SOIC-8_3.9x4.9mm_P1.27mm, symbol HybotixParts:24C32_EEPROM
Other:
- note added: "RPi5 INTERFACE NOTES:\nJ_GPIO40: 40-pin 2x20 2.54mm (RPi5 compatible)\n Pins 1/17: +3V3. Pins 2/4: +5V. Pins 27/28: HAT EEPROM ID_SD/ID_SC\n STM32U585 signals: 3.3V direct\n QRB2210 GPIO: 1.8V → TXS0108E → 3.3V on header\nHAT EEPROM U_EEPROM (24C32 SOIC-8):\n Address 0x50 (A0=A1=A2=GND). Pins 27/28 only.\n 4.7kΩ pullups R_E2/R_E3 to +3V3 on ID_SD/ID_SC\n Program at first boot with RPi HAT EEPROM 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"
- note removed: "RPi5 INTERFACE NOTES: 40-PIN HEADER (J_GPIO40): STM32U585 signals: 3.3V native, direct routing to header QRB2210 MPU GPIO: 1.8V from JMISC → TXS0108E → 3.3V on header Pins 1,17: +3V3 output (from carrier +3V3 rail) Pins 2,4: +5V output (from carrier +5V rail) Pins 27,28: ID_SD/ID_SC — dedicated I2C to HAT ID EEPROM U_EEPROM NO PCIe: QRB2210 has no PCIe root complex — RPi5 NVMe HATs incompatible H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"

Commit message: REBUILD: Minimal KiCad 10.0.2 compatible schematic files
Completely rebuilt all 16 schematic files using absolute minimum structure
that KiCad 10.0.2 on macOS will accept:

Root schematics (2 files):
- uno_q_hub75_shield.kicad_sch (7 sheets)
- uno_q_super_carrier.kicad_sch (7 sheets)

Sub-sheets (14 files):
- All 7 shield sub-sheets
- All 7 carrier sub-sheets

Format: Minimal valid structure — only mandatory elements
- (kicad_sch version 20260326)
- (generator eeschema, generator_version 10.0.0)
- (uuid) for each file
- (lib_symbols) empty section
- (sheet) blocks with uuid + instances
- (sheet_instances) at end
- Hierarchical labels with uuid

No complex symbol instances, no wires, no graphic elements —
just the bare structure KiCad needs to load the files.
Parts:
- removed J_CSI0: CSI0_RPi5_22pin, Connector_FFC-FPC:Molex_503480-2200_1x22-1MP_P0.50mm_Horizontal, symbol HybotixParts:FPC_22pin_0.5mm
- removed J_CSI1: CSI1_RPi5_22pin, Connector_FFC-FPC:Molex_503480-2200_1x22-1MP_P0.50mm_Horizontal, symbol HybotixParts:FPC_22pin_0.5mm
- removed J_GPIO40: RPi5_40PIN, Connector_PinHeader_2.54mm:PinHeader_2x20_P2.54mm_Vertical, symbol HybotixParts:GPIO40_RPi5
- removed R_E1: 0Ω DNP A0=A1=A2=GND addr=0x50, Resistor_SMD:R_0402_1005Metric, symbol Device:R
- removed R_E2: 4.7kΩ 1% 0402 ID_SD pullup, Resistor_SMD:R_0402_1005Metric, symbol Device:R
- removed R_E3: 4.7kΩ 1% 0402 ID_SC pullup, Resistor_SMD:R_0402_1005Metric, symbol Device:R
- removed U_EEPROM: 24C32_HAT_ID, Package_SO:SOIC-8_3.9x4.9mm_P1.27mm, symbol HybotixParts:24C32_EEPROM
Other:
- note removed: "RPi5 INTERFACE NOTES:\nJ_GPIO40: 40-pin 2x20 2.54mm (RPi5 compatible)\n Pins 1/17: +3V3. Pins 2/4: +5V. Pins 27/28: HAT EEPROM ID_SD/ID_SC\n STM32U585 signals: 3.3V direct\n QRB2210 GPIO: 1.8V → TXS0108E → 3.3V on header\nHAT EEPROM U_EEPROM (24C32 SOIC-8):\n Address 0x50 (A0=A1=A2=GND). Pins 27/28 only.\n 4.7kΩ pullups R_E2/R_E3 to +3V3 on ID_SD/ID_SC\n Program at first boot with RPi HAT EEPROM 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"
- company: Hybrid RobotiX -> (none)
- title: UNO Q Super Carrier — RPi5 Compatible Interface -> (none)
