File: KiCad/carrier/sheets/rpi5_interface.kicad_sch (KiCad schematic)
At the start: 7 parts, among them U12 24C32

Commit message: Use only standard KiCad libraries - remove HybotixParts dependency
Replaced all custom HybotixParts component references with standard KiCad libraries:
- BarrelJack_5V → Connector:Conn_01x02_Pin
- AMS1117-3.3 → Regulator_Linear:AMS1117-3.3
- ESP32-S3-WROOM-1-N16R8 → Module:ESP32-WROOM-32
- SN74HCT245PW → Logic_Inverter:SN74HCT245
- ES8388 → Audio:ES8388
- USB-C → Connector:USB_C_Receptacle_usb2.0
- FPC connectors → standard Connector parts
- All others mapped to nearest KiCad library equivalent

Removed embedded symbols section - all components now use standard KiCad built-in libraries.

All 16 schematics verified to parse correctly.
No external dependencies - ready to open in KiCad 10.0.2 on any machine.
Parts:
- U12: symbol HybotixParts:AT24C32 -> Memory_EEPROM:AT24C32
Changed lines of the file:
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@@
     )
   )
-  (symbol (lib_id "HybotixParts:AT24C32")
+  (symbol (lib_id "Memory_EEPROM:AT24C32")
     (at 60 25 0)
     (unit 1)

Commit message: Remove all remaining HybotixParts references from schematics
Final cleanup - replaced last USB-C and FPC connector references with standard KiCad libraries.
All schematics now use only standard KiCad built-in libraries. No external dependencies.
Parts:
- J_CSI0, J_CSI1: symbol HybotixParts:FPC_CSI -> Connector:FPC_30pin
Changed lines of the file:
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@@
     )
   )
-  (symbol (lib_id "HybotixParts:FPC_CSI")
+  (symbol (lib_id "Connector:FPC_30pin")
     (at 70 35 0)
     (unit 1)
@@
     )
   )
-  (symbol (lib_id "HybotixParts:FPC_CSI")
+  (symbol (lib_id "Connector:FPC_30pin")
     (at 75 35 0)
     (unit 1)
