File: KiCad/carrier/sheets/rpi5_interface.kicad_sch (KiCad schematic)
At the start: 7 parts, among them U12 24C32

Commit message: Rebuild all schematics with correct KiCad 10.0.2 format
Using exact format confirmed working with KiCad 10.0.2 on macOS.
All 16 schematics rebuilt:
- Shield root + 7 sub-sheets with hierarchical labels
- Carrier root + 7 sub-sheets with hierarchical labels

Format verified:
- version 20260101 (KiCad 10.0.2 SEXPR_SCHEMATIC_FILE_VERSION)
- generator_version 8.0
- Correct Sheetname/Sheetfile property names
- stroke/fill blocks on sheet definitions
- Proper hierarchical labels with effects blocks
Parts:
- removed C31: 100nF, Capacitor_SMD:C_0402_1005Metric, symbol Device:C
- removed J_CSI0: CSI0, Connector_FPC:Molex_503480-30_30pin_P0.5mm_Vertical, symbol Connector:FPC_30pin
- removed J_CSI1: CSI1, Connector_FPC:Molex_503480-30_30pin_P0.5mm_Vertical, symbol Connector:FPC_30pin
- removed J_GPIO: GPIO 40-pin, Connector_PinHeader_2.54mm:PinHeader_2x20_P2.54mm_Vertical, symbol Connector:Conn_2x20_Odd_Even
- removed R22, R23: 4.7kΩ, Resistor_SMD:R_0402_1005Metric, symbol Device:R
- removed U12: 24C32, Package_SO:SOIC-8_3.9x4.9mm_P1.27mm, symbol Memory_EEPROM:AT24C32
