File: KiCad/carrier/sheets/uno_q_mounting.kicad_sch (KiCad schematic)
At the start: 2 parts

Commit message: REBUILD: Minimal KiCad 10.0.2 compatible schematic files
Completely rebuilt all 16 schematic files using absolute minimum structure
that KiCad 10.0.2 on macOS will accept:

Root schematics (2 files):
- uno_q_hub75_shield.kicad_sch (7 sheets)
- uno_q_super_carrier.kicad_sch (7 sheets)

Sub-sheets (14 files):
- All 7 shield sub-sheets
- All 7 carrier sub-sheets

Format: Minimal valid structure — only mandatory elements
- (kicad_sch version 20260326)
- (generator eeschema, generator_version 10.0.0)
- (uuid) for each file
- (lib_symbols) empty section
- (sheet) blocks with uuid + instances
- (sheet_instances) at end
- Hierarchical labels with uuid

No complex symbol instances, no wires, no graphic elements —
just the bare structure KiCad needs to load the files.
Parts:
- removed B1: JMISC_FTSH-130-01, Connector_PinHeader_1.27mm:PinHeader_2x30_P1.27mm_SMD, symbol HybotixParts:FTSH_130_01
- removed B2: JMEDIA_FTSH-130-01, Connector_PinHeader_1.27mm:PinHeader_2x30_P1.27mm_SMD, symbol HybotixParts:FTSH_130_01
Other:
- note removed: "B1 JMISC / B2 JMEDIA: Samtec FTSH-130-01-L-DV-A\n2x30 contacts 1.27mm pitch SMD mezzanine\nENIG finish required. Placement accuracy ±0.05mm.\nMPU GPIO 1.8V from JMISC → TXS0108E → 3.3V for header/GPIO\nMIPI differential: 100Ω, length-matched, inner layer routing"
- company: Hybrid RobotiX -> (none)
- title: UNO Q Super Carrier — UNO Q Mounting Connectors -> (none)
Changed lines of the file:
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@@
 (kicad_sch
   (version 20260326)
-  (generator "eeschema")
+  (generator eeschema)
   (generator_version "10.0.0")
-  (paper "A3")
-  (title_block
-    (title "UNO Q Super Carrier — UNO Q Mounting Connectors")
-    (date "2026-05-08")
-    (rev "0.1")
-    (company "Hybrid RobotiX")
-    (comment 1 "B1: JMISC (Samtec FTSH-130-01 2x30 1.27mm) SPI I2C GPIO power")
-    (comment 2 "B2: JMEDIA (Samtec FTSH-130-01 2x30 1.27mm) MIPI DSI CSI0 CSI1")
-    (comment 3 "ENIG finish required for 1.27mm pitch SMD mezzanine")
-    (comment 4 "MPU GPIO 1.8V: route to TXS0108E level shifters")
-  )
-  (symbol (lib_id "HybotixParts:FTSH_130_01")
-    (at 80 80 0)
-    (unit 1)
-    (in_bom yes) (on_board yes)
-    (property "Reference" "B1" (at 82 79 0)
-      (effects (font (size 1.27 1.27)))
-    )
-    (property "Value" "JMISC_FTSH-130-01" (at 82 81 0)
-      (effects (font (size 1.27 1.27)))
-    )
-    (property "Footprint" "Connector_PinHeader_1.27mm:PinHeader_2x30_P1.27mm_SMD" (at 80 80 0)
-      (effects (font (size 1.27 1.27)) hide)
-    )
-    (property "Datasheet" "https://suddendocs.samtec.com/prints/ftsh-1xx-xx-xxx-dv-xxx-tr-mkt.pdf" (at 80 80 0)
-      (effects (font (size 1.27 1.27)) hide)
-    )
-    (property "MPN" "FTSH-130-01-L-DV-A" (at 80 80 0)
-      (effects (font (size 1.27 1.27)) hide)
-    )
-    (instances
-      (project "uno_q_super_carrier"
-        (path "/a7d62ed3-8e95-4e64-b6df-722c91664a1a/449d30f0-eb84-4d63-9d19-34540df21399"
-          (reference "B1")
-          (unit 1)
-        )
-      )
+  (paper "A4")
+  (sheet_instances
+    (path "/"
+      (page "1")
     )
   )
-  (symbol (lib_id "HybotixParts:FTSH_130_01")
-    (at 160 80 0)
-    (unit 1)
-    (in_bom yes) (on_board yes)
-    (property "Reference" "B2" (at 162 79 0)
-      (effects (font (size 1.27 1.27)))
-    )
-    (property "Value" "JMEDIA_FTSH-130-01" (at 162 81 0)
-      (effects (font (size 1.27 1.27)))
-    )
-    (property "Footprint" "Connector_PinHeader_1.27mm:PinHeader_2x30_P1.27mm_SMD" (at 160 80 0)
-      (effects (font (size 1.27 1.27)) hide)
-    )
-    (property "Datasheet" "https://suddendocs.samtec.com/prints/ftsh-1xx-xx-xxx-dv-xxx-tr-mkt.pdf" (at 160 80 0)
-      (effects (font (size 1.27 1.27)) hide)
-    )
-    (property "MPN" "FTSH-130-01-L-DV-A" (at 160 80 0)
-      (effects (font (size 1.27 1.27)) hide)
-    )
-    (instances
-      (project "uno_q_super_carrier"
-        (path "/a7d62ed3-8e95-4e64-b6df-722c91664a1a/449d30f0-eb84-4d63-9d19-34540df21399"
-          (reference "B2")
-          (unit 1)
-        )
-      )
-    )
-  )
-  (hierarchical_label "SPI_MOSI"
-    (shape output)
-    (at 50 62 0)
-    (effects (font (size 1.27 1.27)) (justify right))
-  )
-  (hierarchical_label "SPI_MISO"
-    (shape input)
-    (at 50 66 0)
-    (effects (font (size 1.27 1.27)) (justify right))
-  )
-  (hierarchical_label "SPI_SCK"
-    (shape output)
-    (at 50 70 0)
-    (effects (font (size 1.27 1.27)) (justify right))
-  )
-  (hierarchical_label "CS_S3_MCU"
-    (shape output)
-    (at 50 74 0)
-    (effects (font (size 1.27 1.27)) (justify right))
-  )
-  (hierarchical_label "CS_S3_MPU"
-    (shape output)
-    (at 50 78 0)
-    (effects (font (size 1.27 1.27)) (justify right))
-  )
-  (hierarchical_label "CS_C6_MCU"
-    (shape output)
-    (at 50 82 0)
-    (effects (font (size 1.27 1.27)) (justify right))
-  )
-  (hierarchical_label "CS_C6_MPU"
-    (shape output)
-    (at 50 86 0)
-    (effects (font (size 1.27 1.27)) (justify right))
-  )
-  (hierarchical_label "I2C_SDA"
-    (shape bidirectional)
-    (at 50 90 0)
-    (effects (font (size 1.27 1.27)) (justify right))
-  )
-  (hierarchical_label "I2C_SCL"
-    (shape output)
-    (at 50 94 0)
-    (effects (font (size 1.27 1.27)) (justify right))
-  )
-  (hierarchical_label "MPU_GPIO_1V8_BUS"
-    (shape output)
-    (at 110 62 0)
-    (effects (font (size 1.27 1.27)) (justify right))
-  )
-  (hierarchical_label "MPU_1V8_REF"
-    (shape output)
-    (at 110 66 0)
-    (effects (font (size 1.27 1.27)) (justify right))
-  )
-  (hierarchical_label "DSI_CLK_P"
-    (shape output)
-    (at 190 62 0)
-    (effects (font (size 1.27 1.27)) (justify right))
-  )
-  (hierarchical_label "DSI_CLK_N"
-    (shape output)
-    (at 190 66 0)
-    (effects (font (size 1.27 1.27)) (justify right))
-  )
-  (hierarchical_label "DSI_D0_P"
-    (shape output)
-    (at 190 70 0)
-    (effects (font (size 1.27 1.27)) (justify right))
-  )
-  (hierarchical_label "DSI_D0_N"
-    (shape output)
-    (at 190 74 0)
-    (effects (font (size 1.27 1.27)) (justify right))
-  )
-  (hierarchical_label "DSI_D1_P"
-    (shape output)
-    (at 190 78 0)
-    (effects (font (size 1.27 1.27)) (justify right))
-  )
-  (hierarchical_label "DSI_D1_N"
-    (shape output)
-    (at 190 82 0)
-    (effects (font (size 1.27 1.27)) (justify right))
-  )
-  (hierarchical_label "CSI0_CLK_P"
-    (shape output)
-    (at 190 88 0)
-    (effects (font (size 1.27 1.27)) (justify right))
-  )
-  (hierarchical_label "CSI0_CLK_N"
-    (shape output)
-    (at 190 92 0)
-    (effects (font (size 1.27 1.27)) (justify right))
-  )
-  (hierarchical_label "CSI1_CLK_P"
-    (shape output)
-    (at 190 96 0)
-    (effects (font (size 1.27 1.27)) (justify right))
-  )
-  (hierarchical_label "CSI1_CLK_N"
-    (shape output)
-    (at 190 100 0)
-    (effects (font (size 1.27 1.27)) (justify right))
-  )
-  (text "B1 JMISC / B2 JMEDIA: Samtec FTSH-130-01-L-DV-A\\n2x30 contacts 1.27mm pitch SMD mezzanine\\nENIG finish required. Placement accuracy ±0.05mm.\\nMPU GPIO 1.8V from JMISC → TXS0108E → 3.3V for header/GPIO\\nMIPI differential: 100Ω, length-matched, inner layer routing"
-    (at 20 130 0)
-    (effects (font (size 1.27 1.27)) (justify left top))
-  )
-  (sheet_instances
-    (path "/"
-      (page "3")
-    )
-  )
