File: KiCad/carrier/sheets/uno_q_mounting.kicad_sch (KiCad schematic)
At the start: 0 parts

Commit message: Add carrier schematic generator + rebuild all carrier schematics with complete BOM
Generator:
- build_carrier_complete.py: Carrier-specific generator with all 7 sheets + root

Carrier rebuilt with complete component list from BOM:
- power.kicad_sch: TPS54331 buck, dual VIN support, feedback divider (13 components)
- uno_q_mounting.kicad_sch: Samtec FTSH-130-01 mezzanine connectors (2 components + power/signals)
- esp32c6_radio.kicad_sch: ESP32-C6-MINI-1 module, antenna selection, U.FL connector (6 components)
- display_chain.kicad_sch: LT8618SX MIPI→HDMI, CBTL04GP054 switch, Micro-HDMI (5 components)
- rpi5_interface.kicad_sch: 40-pin GPIO, 24C32 HAT EEPROM, CSI0/CSI1 FPC (8 components)
- level_shift.kicad_sch: TXS0108E x2 level shifters for MPU GPIO (2 components)
- expansion.kicad_sch: Qwiic x2, Grove x5 with pullups (7 components)
- uno_q_super_carrier.kicad_sch: Root schematic with all 7 sheets

All 8 files verified with kicad-skip parser (KiCad 10.0.2 compatible).
Regenerable from scripts - ready to open in KiCad 10.0.2.
Parts:
- added B1: JMISC, Connector_Samtec:Samtec_FTSH-130-01-L-DV-A_2x30_P1.27mm_Vertical, symbol HybotixParts:FTSH-130-01
- added B2: JMEDIA, Connector_Samtec:Samtec_FTSH-130-01-L-DV-A_2x30_P1.27mm_Vertical, symbol HybotixParts:FTSH-130-01
Changed lines of the file:
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@@
   (generator_version "10.0.0")
   (paper "A4")
+  (symbol (lib_id "HybotixParts:FTSH-130-01")
+    (at 30 25 0)
+    (unit 1)
+    (in_bom yes) (on_board yes)
+    (property "Reference" "B1"
+      (at 30 23.5 0)
+      (effects (font (size 1.27 1.27)))
+    )
+    (property "Value" "JMISC"
+      (at 30 26.5 0)
+      (effects (font (size 1.27 1.27)))
+    )
+    (property "Footprint" "Connector_Samtec:Samtec_FTSH-130-01-L-DV-A_2x30_P1.27mm_Vertical"
+      (at 30 25 0)
+      (effects (font (size 1.27 1.27)) hide)
+    )
+    (instances
+      (project "uno_q_hub75_shield"
+        (path "/bc84562d-846a-4607-81a1-500b7991d137/SHEETUUID"
+          (reference "B1") (unit 1)
+        )
+      )
+    )
+  )
+  (symbol (lib_id "HybotixParts:FTSH-130-01")
+    (at 50 25 0)
+    (unit 1)
+    (in_bom yes) (on_board yes)
+    (property "Reference" "B2"
+      (at 50 23.5 0)
+      (effects (font (size 1.27 1.27)))
+    )
+    (property "Value" "JMEDIA"
+      (at 50 26.5 0)
+      (effects (font (size 1.27 1.27)))
+    )
+    (property "Footprint" "Connector_Samtec:Samtec_FTSH-130-01-L-DV-A_2x30_P1.27mm_Vertical"
+      (at 50 25 0)
+      (effects (font (size 1.27 1.27)) hide)
+    )
+    (instances
+      (project "uno_q_hub75_shield"
+        (path "/bc84562d-846a-4607-81a1-500b7991d137/SHEETUUID"
+          (reference "B2") (unit 1)
+        )
+      )
+    )
+  )
+  (hierarchical_label "+5V"
+    (shape input)
+    (at 10 20 0)
+    (effects (font (size 1.27 1.27)) (justify left))
+  )
+  (hierarchical_label "+3V3"
+    (shape input)
+    (at 10 25 0)
+    (effects (font (size 1.27 1.27)) (justify left))
+  )
+  (hierarchical_label "DGND"
+    (shape input)
+    (at 10 30 0)
+    (effects (font (size 1.27 1.27)) (justify left))
+  )
+  (hierarchical_label "CS_S3_MPU"
+    (shape input)
+    (at 10 40 0)
+    (effects (font (size 1.27 1.27)) (justify left))
+  )
+  (hierarchical_label "S3_C6_TX"
+    (shape output)
+    (at 70 20 0)
+    (effects (font (size 1.27 1.27)) (justify left))
+  )
+  (hierarchical_label "S3_C6_RX"
+    (shape input)
+    (at 70 25 0)
+    (effects (font (size 1.27 1.27)) (justify left))
+  )
   (sheet_instances
     (path "/"
