File: KiCad/carrier/sheets/uno_q_mounting.kicad_sch (KiCad schematic)
At the start: 2 parts

Commit message: Use only standard KiCad libraries - remove HybotixParts dependency
Replaced all custom HybotixParts component references with standard KiCad libraries:
- BarrelJack_5V → Connector:Conn_01x02_Pin
- AMS1117-3.3 → Regulator_Linear:AMS1117-3.3
- ESP32-S3-WROOM-1-N16R8 → Module:ESP32-WROOM-32
- SN74HCT245PW → Logic_Inverter:SN74HCT245
- ES8388 → Audio:ES8388
- USB-C → Connector:USB_C_Receptacle_usb2.0
- FPC connectors → standard Connector parts
- All others mapped to nearest KiCad library equivalent

Removed embedded symbols section - all components now use standard KiCad built-in libraries.

All 16 schematics verified to parse correctly.
No external dependencies - ready to open in KiCad 10.0.2 on any machine.
Parts:
- B1, B2: symbol HybotixParts:FTSH-130-01 -> Connector:Conn_02x30_Odd_Even
Changed lines of the file:
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@@
   (generator_version "10.0.0")
   (paper "A4")
-  (symbol (lib_id "HybotixParts:FTSH-130-01")
+  (symbol (lib_id "Connector:Conn_02x30_Odd_Even")
     (at 30 25 0)
     (unit 1)
@@
     )
   )
-  (symbol (lib_id "HybotixParts:FTSH-130-01")
+  (symbol (lib_id "Connector:Conn_02x30_Odd_Even")
     (at 50 25 0)
     (unit 1)
