File: KiCad/carrier/sheets/power.kicad_sch (KiCad schematic)
At the start: 11 parts, among them U7 TPS54331DR, U8 AMS1117-3.3

Commit message: Rebuild all schematics with correct KiCad 10.0.2 format
Using exact format confirmed working with KiCad 10.0.2 on macOS.
All 16 schematics rebuilt:
- Shield root + 7 sub-sheets with hierarchical labels
- Carrier root + 7 sub-sheets with hierarchical labels

Format verified:
- version 20260101 (KiCad 10.0.2 SEXPR_SCHEMATIC_FILE_VERSION)
- generator_version 8.0
- Correct Sheetname/Sheetfile property names
- stroke/fill blocks on sheet definitions
- Proper hierarchical labels with effects blocks
Parts:
- removed C18, C19, C22: 100µF, Capacitor_SMD:C_1206_3216Metric, symbol Device:C
- removed C23, C26: 100nF, Capacitor_SMD:C_0402_1005Metric, symbol Device:C
- removed C24: 4.7µF, Capacitor_SMD:C_0805_2012Metric, symbol Device:C
- removed C25: 10µF, Capacitor_SMD:C_0805_2012Metric, symbol Device:C
- removed R_P1, R_P2: 100kΩ, Resistor_SMD:R_0402_1005Metric, symbol Device:R
- removed U7: TPS54331DR, Package_SO:SOIC-8_3.9x4.9mm_P1.27mm, symbol Regulator_Switching:TPS54331
- removed U8: AMS1117-3.3, Package_TO_SOT_SMD:SOT-223-3_TabPin2, symbol Regulator_Linear:AMS1117-3.3
