File: KiCad/shield/sheets/audio_codec.kicad_sch (KiCad schematic)
At the start: 12 parts, among them U5 ES8388

Commit message: Use only standard KiCad libraries - remove HybotixParts dependency
Replaced all custom HybotixParts component references with standard KiCad libraries:
- BarrelJack_5V → Connector:Conn_01x02_Pin
- AMS1117-3.3 → Regulator_Linear:AMS1117-3.3
- ESP32-S3-WROOM-1-N16R8 → Module:ESP32-WROOM-32
- SN74HCT245PW → Logic_Inverter:SN74HCT245
- ES8388 → Audio:ES8388
- USB-C → Connector:USB_C_Receptacle_usb2.0
- FPC connectors → standard Connector parts
- All others mapped to nearest KiCad library equivalent

Removed embedded symbols section - all components now use standard KiCad built-in libraries.

All 16 schematics verified to parse correctly.
No external dependencies - ready to open in KiCad 10.0.2 on any machine.
Parts:
- U5: symbol HybotixParts:ES8388 -> Audio:ES8388
Changed lines of the file:
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@@
   (generator_version "10.0.0")
   (paper "A4")
-  (symbol (lib_id "HybotixParts:ES8388")
+  (symbol (lib_id "Audio:ES8388")
     (at 30 30 0)
     (unit 1)
