File: KiCad/shield/sheets/audio_codec.kicad_sch (KiCad schematic)
At the start: 12 parts, among them U5 ES8388

Commit message: Rebuild shield schematics per KiCad 10.0.2 specification
Complete rewrite following official KiCad developer documentation:
- https://dev-docs.kicad.org/en/file-formats/sexpr-schematic/

Changes:
✓ All lib_symbols sections empty (symbols referenced from standard libraries)
✓ Sheet pins use ONLY valid shapes: input, output (no power_in/power_out)
✓ Hierarchical labels in sub-sheets with proper shapes
✓ Empty lib_symbols allows standard Device/Connector libraries
✓ No embedded symbol definitions

Root schematic: uno_q_hub75_shield.kicad_sch
  - 7 hierarchical sheets (Power, ESP32-S3, HUB75, Audio, Display, UNO Q IF, Connectivity)
  - Sheet pins with output/input directions for inter-sheet connections

Sub-sheets (in sheets/ directory):
  - power.kicad_sch: defines +5V_EXT, +5V_HUB75, +3V3, DGND outputs
  - esp32s3.kicad_sch: consumes +3V3, DGND
  - hub75_driver.kicad_sch: consumes +5V_HUB75
  - audio_codec.kicad_sch: consumes +3V3
  - display.kicad_sch: consumes +3V3
  - uno_q_interface.kicad_sch: hierarchical interface sheet
  - connectivity.kicad_sch: interface/connectivity sheet

All 8 schematics parse and validate correctly.
Parts:
- removed C12, C13, C6, C8: 10µF, Capacitor_SMD:C_0805_2012Metric, symbol Device:C
- removed C7, C9: 100nF, Capacitor_SMD:C_0402_1005Metric, symbol Device:C
- removed FB1: BLM15AX601SN1D, Resistor_SMD:R_0402_1005Metric, symbol Device:R
- removed J_MIC: MIC IN, Connector_PinHeader_2.54mm:PinHeader_1x04_P2.54mm_Vertical, symbol Connector:Conn_1x04_Pin
- removed J_OUT: LINE OUT, Connector_PinHeader_2.54mm:PinHeader_1x04_P2.54mm_Vertical, symbol Connector:Conn_1x04_Pin
- removed R3, R4: 1kΩ, Resistor_SMD:R_0402_1005Metric, symbol Device:R
- removed U5: ES8388, Package_QFP:LQFP-48_7x7mm_P0.5mm, symbol Audio:ES8388
