File: KiCad/shield/sheets/connectivity.kicad_sch (KiCad schematic)
At the start: 9 parts, among them J10 Grove, J11 Grove, J12 Grove, J13 Grove, J14 Grove, J8 Qwiic, J9 Qwiic

Commit message: Use only standard KiCad libraries - remove HybotixParts dependency
Replaced all custom HybotixParts component references with standard KiCad libraries:
- BarrelJack_5V → Connector:Conn_01x02_Pin
- AMS1117-3.3 → Regulator_Linear:AMS1117-3.3
- ESP32-S3-WROOM-1-N16R8 → Module:ESP32-WROOM-32
- SN74HCT245PW → Logic_Inverter:SN74HCT245
- ES8388 → Audio:ES8388
- USB-C → Connector:USB_C_Receptacle_usb2.0
- FPC connectors → standard Connector parts
- All others mapped to nearest KiCad library equivalent

Removed embedded symbols section - all components now use standard KiCad built-in libraries.

All 16 schematics verified to parse correctly.
No external dependencies - ready to open in KiCad 10.0.2 on any machine.
Parts:
- J10, J11, J12, J13, J14: symbol HybotixParts:Grove_4pin -> Connector:Conn_01x04_Pin
- J8, J9: symbol HybotixParts:Qwiic_JST_SH_4 -> Connector:Conn_01x04_Pin
Changed lines of the file:
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@@
   (generator_version "10.0.0")
   (paper "A4")
-  (symbol (lib_id "HybotixParts:Qwiic_JST_SH_4")
+  (symbol (lib_id "Connector:Conn_01x04_Pin")
     (at 30 20 0)
     (unit 1)
@@
     )
   )
-  (symbol (lib_id "HybotixParts:Qwiic_JST_SH_4")
+  (symbol (lib_id "Connector:Conn_01x04_Pin")
     (at 40 20 0)
     (unit 1)
@@
     )
   )
-  (symbol (lib_id "HybotixParts:Grove_4pin")
+  (symbol (lib_id "Connector:Conn_01x04_Pin")
     (at 30 40 0)
     (unit 1)
@@
     )
   )
-  (symbol (lib_id "HybotixParts:Grove_4pin")
+  (symbol (lib_id "Connector:Conn_01x04_Pin")
     (at 40 40 0)
     (unit 1)
@@
     )
   )
-  (symbol (lib_id "HybotixParts:Grove_4pin")
+  (symbol (lib_id "Connector:Conn_01x04_Pin")
     (at 50 40 0)
     (unit 1)
@@
     )
   )
-  (symbol (lib_id "HybotixParts:Grove_4pin")
+  (symbol (lib_id "Connector:Conn_01x04_Pin")
     (at 60 40 0)
     (unit 1)
@@
     )
   )
-  (symbol (lib_id "HybotixParts:Grove_4pin")
+  (symbol (lib_id "Connector:Conn_01x04_Pin")
     (at 70 40 0)
     (unit 1)
