File: KiCad/shield/sheets/connectivity.kicad_sch (KiCad schematic)
At the start: 0 parts

Commit message: Populate shield schematics with actual components from BOM/DESIGN_SPEC
Power sheet: J4 barrel jack, C1/C2 bulk+bypass, U4 AMS1117-3.3,
  C3-C5 regulator caps, D1/D2 LEDs, R1/R2 current limiters

ESP32-S3 sheet: U1 ESP32-S3-WROOM-1-N16R8, R10/R11 pullups,
  C10/C11 bypass, J5 USB-C, R12/R13 CC resistors,
  All 20 GPIO hierarchical labels connected

HUB75 Driver: U2/U3 SN74HCT245PW level shifters, J1 HUB75 IDC,
  C16/C17 bypass caps, 0R DIR/OE ties to GND

Audio Codec: U5 ES8388, FB1 ferrite, C6-C9 supply caps,
  R3/R4 I2C pullups, C12-C15 DC blocking, J_OUT/J_MIC headers

Display: J6 Molex 503480-2200 22-pin FPC, R20/R21 GT911 pullups,
  C20/C21 bypass caps, JP1 SPI mode select

UNO Q Interface: J2 SPI header, J3 debug UART header

Connectivity: J8/J9 Qwiic, R5/R6 pullups, J10-J14 Grove connectors
Parts:
- added J10: Grove_I2C, Connector_Grove:Grove_4P-2.00mm, symbol Connector:Conn_01x04_Pin
- added J11: Grove_UART, Connector_Grove:Grove_4P-2.00mm, symbol Connector:Conn_01x04_Pin
- added J12: Grove_SPI, Connector_Grove:Grove_4P-2.00mm, symbol Connector:Conn_01x04_Pin
- added J13: Grove_Digital, Connector_Grove:Grove_4P-2.00mm, symbol Connector:Conn_01x04_Pin
- added J14: Grove_Analog, Connector_Grove:Grove_4P-2.00mm, symbol Connector:Conn_01x04_Pin
- added J8: Qwiic_1, Connector_JST:JST_SH_SM04B-SRSS-TB_1x04-1MP_P1.00mm_Horizontal, symbol Connector:Conn_01x04_Pin
- added J9: Qwiic_2, Connector_JST:JST_SH_SM04B-SRSS-TB_1x04-1MP_P1.00mm_Horizontal, symbol Connector:Conn_01x04_Pin
- added R5, R6: 4.7k, Resistor_SMD:R_0402_1005Metric, symbol Device:R
Changed lines of the file:
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@@
 	(generator_version "8.0")
 	(paper "A4")
-	(hierarchical_label "+3V3"
-		(shape input)
-		(at 10 25 0)
-		(fields_autoplaced yes)
-		(effects
-			(font
-				(size 1.27 1.27)
-			)
-			(justify left)
-		)
-		(uuid "5d6e7f8a-9b0c-1d2e-3f4a-5b6c7d8e9f0a-hl00")
-	)
-	(hierarchical_label "I2C_SDA"
-		(shape bidirectional)
-		(at 10 30 0)
-		(fields_autoplaced yes)
-		(effects
-			(font
-				(size 1.27 1.27)
-			)
-			(justify left)
-		)
-		(uuid "5d6e7f8a-9b0c-1d2e-3f4a-5b6c7d8e9f0a-hl01")
-	)
-	(hierarchical_label "I2C_SCL"
-		(shape bidirectional)
-		(at 10 35 0)
-		(fields_autoplaced yes)
-		(effects
-			(font
-				(size 1.27 1.27)
-			)
-			(justify left)
-		)
-		(uuid "5d6e7f8a-9b0c-1d2e-3f4a-5b6c7d8e9f0a-hl02")
-	)
+  (hierarchical_label "+3V3"
+    (shape input)
+    (at 10 20 0)
+    (fields_autoplaced yes)
+    (effects (font (size 1.27 1.27)) (justify left))
+    (uuid "hl-conn-3v3-in")
+  )
+  (hierarchical_label "DGND"
+    (shape input)
+    (at 10 25 0)
+    (fields_autoplaced yes)
+    (effects (font (size 1.27 1.27)) (justify left))
+    (uuid "hl-conn-dgnd-in")
+  )
+  (hierarchical_label "I2C_SDA"
+    (shape bidirectional)
+    (at 10 40 0)
+    (fields_autoplaced yes)
+    (effects (font (size 1.27 1.27)) (justify left))
+    (uuid "hl-conn-sda")
+  )
+  (hierarchical_label "I2C_SCL"
+    (shape bidirectional)
+    (at 10 45 0)
+    (fields_autoplaced yes)
+    (effects (font (size 1.27 1.27)) (justify left))
+    (uuid "hl-conn-scl")
+  )
+  (symbol (lib_id "Connector:Conn_01x04_Pin")
+    (at 60 40 0)
+    (unit 1)
+    (in_bom yes) (on_board yes)
+    (uuid "j8-uuid")
+    (property "Reference" "J8" (at 62 38 0) (effects (font (size 1.27 1.27))))
+    (property "Value" "Qwiic_1" (at 62 42 0) (effects (font (size 1.27 1.27))))
+    (property "Footprint" "Connector_JST:JST_SH_SM04B-SRSS-TB_1x04-1MP_P1.00mm_Horizontal" (at 60 40 0) (effects (font (size 1.27 1.27)) (hide yes)))
+    (instances (project "uno_q_hub75_shield" (path "/bc84562d-846a-4607-81a1-500b7991d137/{}" (reference "J8") (unit 1))))
+  )
+  (symbol (lib_id "Connector:Conn_01x04_Pin")
+    (at 60 55 0)
+    (unit 1)
+    (in_bom yes) (on_board yes)
+    (uuid "j9-uuid")
+    (property "Reference" "J9" (at 62 53 0) (effects (font (size 1.27 1.27))))
+    (property "Value" "Qwiic_2" (at 62 57 0) (effects (font (size 1.27 1.27))))
+    (property "Footprint" "Connector_JST:JST_SH_SM04B-SRSS-TB_1x04-1MP_P1.00mm_Horizontal" (at 60 55 0) (effects (font (size 1.27 1.27)) (hide yes)))
+    (instances (project "uno_q_hub75_shield" (path "/bc84562d-846a-4607-81a1-500b7991d137/{}" (reference "J9") (unit 1))))
+  )
+  (symbol (lib_id "Device:R")
+    (at 45 40 90)
+    (unit 1)
+    (in_bom yes) (on_board yes)
+    (uuid "r5-uuid")
+    (property "Reference" "R5" (at 47 38 0) (effects (font (size 1.27 1.27))))
+    (property "Value" "4.7k" (at 47 42 0) (effects (font (size 1.27 1.27))))
+    (property "Footprint" "Resistor_SMD:R_0402_1005Metric" (at 45 40 0) (effects (font (size 1.27 1.27)) (hide yes)))
+    (instances (project "uno_q_hub75_shield" (path "/bc84562d-846a-4607-81a1-500b7991d137/{}" (reference "R5") (unit 1))))
+  )
+  (symbol (lib_id "Device:R")
+    (at 53 40 90)
+    (unit 1)
+    (in_bom yes) (on_board yes)
+    (uuid "r6-uuid")
+    (property "Reference" "R6" (at 55 38 0) (effects (font (size 1.27 1.27))))
+    (property "Value" "4.7k" (at 55 42 0) (effects (font (size 1.27 1.27))))
+    (property "Footprint" "Resistor_SMD:R_0402_1005Metric" (at 53 40 0) (effects (font (size 1.27 1.27)) (hide yes)))
+    (instances (project "uno_q_hub75_shield" (path "/bc84562d-846a-4607-81a1-500b7991d137/{}" (reference "R6") (unit 1))))
+  )
+  (symbol (lib_id "Connector:Conn_01x04_Pin")
+    (at 60 70 0)
+    (unit 1)
+    (in_bom yes) (on_board yes)
+    (uuid "j10-uuid")
+    (property "Reference" "J10" (at 62 68 0) (effects (font (size 1.27 1.27))))
+    (property "Value" "Grove_I2C" (at 62 72 0) (effects (font (size 1.27 1.27))))
+    (property "Footprint" "Connector_Grove:Grove_4P-2.00mm" (at 60 70 0) (effects (font (size 1.27 1.27)) (hide yes)))
+    (instances (project "uno_q_hub75_shield" (path "/bc84562d-846a-4607-81a1-500b7991d137/{}" (reference "J10") (unit 1))))
+  )
+  (symbol (lib_id "Connector:Conn_01x04_Pin")
+    (at 60 82 0)
+    (unit 1)
+    (in_bom yes) (on_board yes)
+    (uuid "j11-uuid")
+    (property "Reference" "J11" (at 62 80 0) (effects (font (size 1.27 1.27))))
+    (property "Value" "Grove_UART" (at 62 84 0) (effects (font (size 1.27 1.27))))
+    (property "Footprint" "Connector_Grove:Grove_4P-2.00mm" (at 60 82 0) (effects (font (size 1.27 1.27)) (hide yes)))
+    (instances (project "uno_q_hub75_shield" (path "/bc84562d-846a-4607-81a1-500b7991d137/{}" (reference "J11") (unit 1))))
+  )
+  (symbol (lib_id "Connector:Conn_01x04_Pin")
+    (at 60 94 0)
+    (unit 1)
+    (in_bom yes) (on_board yes)
+    (uuid "j12-uuid")
+    (property "Reference" "J12" (at 62 92 0) (effects (font (size 1.27 1.27))))
+    (property "Value" "Grove_SPI" (at 62 96 0) (effects (font (size 1.27 1.27))))
+    (property "Footprint" "Connector_Grove:Grove_4P-2.00mm" (at 60 94 0) (effects (font (size 1.27 1.27)) (hide yes)))
+    (instances (project "uno_q_hub75_shield" (path "/bc84562d-846a-4607-81a1-500b7991d137/{}" (reference "J12") (unit 1))))
+  )
+  (symbol (lib_id "Connector:Conn_01x04_Pin")
+    (at 60 106 0)
+    (unit 1)
+    (in_bom yes) (on_board yes)
+    (uuid "j13-uuid")
+    (property "Reference" "J13" (at 62 104 0) (effects (font (size 1.27 1.27))))
+    (property "Value" "Grove_Digital" (at 62 108 0) (effects (font (size 1.27 1.27))))
+    (property "Footprint" "Connector_Grove:Grove_4P-2.00mm" (at 60 106 0) (effects (font (size 1.27 1.27)) (hide yes)))
+    (instances (project "uno_q_hub75_shield" (path "/bc84562d-846a-4607-81a1-500b7991d137/{}" (reference "J13") (unit 1))))
+  )
+  (symbol (lib_id "Connector:Conn_01x04_Pin")
+    (at 60 118 0)
+    (unit 1)
+    (in_bom yes) (on_board yes)
+    (uuid "j14-uuid")
+    (property "Reference" "J14" (at 62 116 0) (effects (font (size 1.27 1.27))))
+    (property "Value" "Grove_Analog" (at 62 120 0) (effects (font (size 1.27 1.27))))
+    (property "Footprint" "Connector_Grove:Grove_4P-2.00mm" (at 60 118 0) (effects (font (size 1.27 1.27)) (hide yes)))
+    (instances (project "uno_q_hub75_shield" (path "/bc84562d-846a-4607-81a1-500b7991d137/{}" (reference "J14") (unit 1))))
+  )
 	(sheet_instances
 		(path "/"
