File: KiCad/shield/sheets/power.kicad_sch (KiCad schematic)
At the start: 13 parts, among them J4 DC +5V IN, U4 AMS1117-3.3

Commit message: Rebuild shield schematics per KiCad 10.0.2 specification
Complete rewrite following official KiCad developer documentation:
- https://dev-docs.kicad.org/en/file-formats/sexpr-schematic/

Changes:
✓ All lib_symbols sections empty (symbols referenced from standard libraries)
✓ Sheet pins use ONLY valid shapes: input, output (no power_in/power_out)
✓ Hierarchical labels in sub-sheets with proper shapes
✓ Empty lib_symbols allows standard Device/Connector libraries
✓ No embedded symbol definitions

Root schematic: uno_q_hub75_shield.kicad_sch
  - 7 hierarchical sheets (Power, ESP32-S3, HUB75, Audio, Display, UNO Q IF, Connectivity)
  - Sheet pins with output/input directions for inter-sheet connections

Sub-sheets (in sheets/ directory):
  - power.kicad_sch: defines +5V_EXT, +5V_HUB75, +3V3, DGND outputs
  - esp32s3.kicad_sch: consumes +3V3, DGND
  - hub75_driver.kicad_sch: consumes +5V_HUB75
  - audio_codec.kicad_sch: consumes +3V3
  - display.kicad_sch: consumes +3V3
  - uno_q_interface.kicad_sch: hierarchical interface sheet
  - connectivity.kicad_sch: interface/connectivity sheet

All 8 schematics parse and validate correctly.
Parts:
- removed C1: 100µF, Capacitor_SMD:C_1206_3216Metric, symbol Device:C
- removed C2, C5: 100nF, Capacitor_SMD:C_0402_1005Metric, symbol Device:C
- removed C3, C4: 10µF, Capacitor_SMD:C_0805_2012Metric, symbol Device:C
- removed D1, D2: Green LED, LED_SMD:LED_0402_1005Metric, symbol Device:LED
- removed J4: DC +5V IN, Connector_BarrelJack:BarrelJack_CUI_PJ-102AH_Horizontal, symbol Connector:Conn_01x02_Pin
- removed R1: 620Ω, Resistor_SMD:R_0402_1005Metric, symbol Device:R
- removed R10, R11: 10kΩ, Resistor_SMD:R_0402_1005Metric, symbol Device:R
- removed R2: 270Ω, Resistor_SMD:R_0402_1005Metric, symbol Device:R
- removed U4: AMS1117-3.3, Package_TO_SOT_SMD:SOT-223-3_TabPin2, symbol Regulator_Linear:AMS1117-3.3
