File: KiCad/shield/sheets/uno_q_interface.kicad_sch (KiCad schematic)
At the start: 2 parts, among them J2 SPI3, J3 UART

Commit message: Rebuild shield schematics per KiCad 10.0.2 specification
Complete rewrite following official KiCad developer documentation:
- https://dev-docs.kicad.org/en/file-formats/sexpr-schematic/

Changes:
✓ All lib_symbols sections empty (symbols referenced from standard libraries)
✓ Sheet pins use ONLY valid shapes: input, output (no power_in/power_out)
✓ Hierarchical labels in sub-sheets with proper shapes
✓ Empty lib_symbols allows standard Device/Connector libraries
✓ No embedded symbol definitions

Root schematic: uno_q_hub75_shield.kicad_sch
  - 7 hierarchical sheets (Power, ESP32-S3, HUB75, Audio, Display, UNO Q IF, Connectivity)
  - Sheet pins with output/input directions for inter-sheet connections

Sub-sheets (in sheets/ directory):
  - power.kicad_sch: defines +5V_EXT, +5V_HUB75, +3V3, DGND outputs
  - esp32s3.kicad_sch: consumes +3V3, DGND
  - hub75_driver.kicad_sch: consumes +5V_HUB75
  - audio_codec.kicad_sch: consumes +3V3
  - display.kicad_sch: consumes +3V3
  - uno_q_interface.kicad_sch: hierarchical interface sheet
  - connectivity.kicad_sch: interface/connectivity sheet

All 8 schematics parse and validate correctly.
Parts:
- removed J2: SPI3, Connector_PinHeader_2.54mm:PinHeader_1x06_P2.54mm_Vertical, symbol Connector:Conn_1x06_Pin
- removed J3: UART, Connector_PinHeader_2.54mm:PinHeader_1x02_P2.54mm_Vertical, symbol Connector:Conn_1x02_Pin
Changed lines of the file:
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@@
   (generator_version "10.0.0")
   (paper "A4")
-  (symbol (lib_id "Connector:Conn_1x06_Pin")
-    (at 30 25 0)
-    (unit 1)
-    (in_bom yes) (on_board yes)
-    (property "Reference" "J2"
-      (at 30 23.5 0)
-      (effects (font (size 1.27 1.27)))
-    )
-    (property "Value" "SPI3"
-      (at 30 26.5 0)
-      (effects (font (size 1.27 1.27)))
-    )
-    (property "Footprint" "Connector_PinHeader_2.54mm:PinHeader_1x06_P2.54mm_Vertical"
-      (at 30 25 0)
-      (effects (font (size 1.27 1.27)) hide)
-    )
-    (instances
-      (project "uno_q_hub75_shield"
-        (path "/bc84562d-846a-4607-81a1-500b7991d137/4c5d6e7f-8a9b-0c1d-2e3f-4a5b6c7d8e9f"
-          (reference "J2") (unit 1)
-        )
-      )
-    )
-  )
-  (symbol (lib_id "Connector:Conn_1x02_Pin")
-    (at 50 25 0)
-    (unit 1)
-    (in_bom yes) (on_board yes)
-    (property "Reference" "J3"
-      (at 50 23.5 0)
-      (effects (font (size 1.27 1.27)))
-    )
-    (property "Value" "UART"
-      (at 50 26.5 0)
-      (effects (font (size 1.27 1.27)))
-    )
-    (property "Footprint" "Connector_PinHeader_2.54mm:PinHeader_1x02_P2.54mm_Vertical"
-      (at 50 25 0)
-      (effects (font (size 1.27 1.27)) hide)
-    )
-    (instances
-      (project "uno_q_hub75_shield"
-        (path "/bc84562d-846a-4607-81a1-500b7991d137/4c5d6e7f-8a9b-0c1d-2e3f-4a5b6c7d8e9f"
-          (reference "J3") (unit 1)
-        )
-      )
-    )
-  )
-  (hierarchical_label "SPI_MOSI"
-    (shape input)
-    (at 10 20 0)
-    (effects (font (size 1.27 1.27)) (justify left))
-  )
-  (hierarchical_label "SPI_MISO"
-    (shape input)
-    (at 10 25 0)
-    (effects (font (size 1.27 1.27)) (justify left))
-  )
-  (hierarchical_label "SPI_SCK"
-    (shape input)
-    (at 10 30 0)
-    (effects (font (size 1.27 1.27)) (justify left))
-  )
-  (hierarchical_label "CS_S3_MCU"
-    (shape input)
-    (at 10 35 0)
-    (effects (font (size 1.27 1.27)) (justify left))
-  )
-  (hierarchical_label "GPIO47"
-    (shape input)
-    (at 10 40 0)
-    (effects (font (size 1.27 1.27)) (justify left))
-  )
   (sheet_instances
-    (path "/"
-      (page "1")
-    )
+    (path "/" (page "7"))
   )
 )
