File: KiCad/shield/sheets/display.kicad_sch (KiCad schematic)
At the start: 4 parts, among them J6 FPC 22-pin

Commit message: Rebuild shield schematics per KiCad 10.0.2 specification
Complete rewrite following official KiCad developer documentation:
- https://dev-docs.kicad.org/en/file-formats/sexpr-schematic/

Changes:
✓ All lib_symbols sections empty (symbols referenced from standard libraries)
✓ Sheet pins use ONLY valid shapes: input, output (no power_in/power_out)
✓ Hierarchical labels in sub-sheets with proper shapes
✓ Empty lib_symbols allows standard Device/Connector libraries
✓ No embedded symbol definitions

Root schematic: uno_q_hub75_shield.kicad_sch
  - 7 hierarchical sheets (Power, ESP32-S3, HUB75, Audio, Display, UNO Q IF, Connectivity)
  - Sheet pins with output/input directions for inter-sheet connections

Sub-sheets (in sheets/ directory):
  - power.kicad_sch: defines +5V_EXT, +5V_HUB75, +3V3, DGND outputs
  - esp32s3.kicad_sch: consumes +3V3, DGND
  - hub75_driver.kicad_sch: consumes +5V_HUB75
  - audio_codec.kicad_sch: consumes +3V3
  - display.kicad_sch: consumes +3V3
  - uno_q_interface.kicad_sch: hierarchical interface sheet
  - connectivity.kicad_sch: interface/connectivity sheet

All 8 schematics parse and validate correctly.
Parts:
- removed J6: FPC 22-pin, Connector_FPC:Molex_503480-2200_22pin_P0.5mm_Vertical, symbol Connector:FPC_22pin_0.5mm
- removed JP1: 0Ω, Resistor_SMD:R_0402_1005Metric, symbol Device:R
- removed R20, R21: 4.7kΩ, Resistor_SMD:R_0402_1005Metric, symbol Device:R
Changed lines of the file:
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@@
   (generator_version "10.0.0")
   (paper "A4")
-  (symbol (lib_id "Connector:FPC_22pin_0.5mm")
-    (at 30 30 0)
-    (unit 1)
-    (in_bom yes) (on_board yes)
-    (property "Reference" "J6"
-      (at 30 28.5 0)
-      (effects (font (size 1.27 1.27)))
-    )
-    (property "Value" "FPC 22-pin"
-      (at 30 31.5 0)
-      (effects (font (size 1.27 1.27)))
-    )
-    (property "Footprint" "Connector_FPC:Molex_503480-2200_22pin_P0.5mm_Vertical"
-      (at 30 30 0)
-      (effects (font (size 1.27 1.27)) hide)
-    )
-    (instances
-      (project "uno_q_hub75_shield"
-        (path "/bc84562d-846a-4607-81a1-500b7991d137/3b4c5d6e-7f8a-9b0c-1d2e-3f4a5b6c7d8e"
-          (reference "J6") (unit 1)
-        )
-      )
-    )
-  )
-  (symbol (lib_id "Device:R")
-    (at 50 25 0)
-    (unit 1)
-    (in_bom yes) (on_board yes)
-    (property "Reference" "R20"
-      (at 50 23.5 0)
-      (effects (font (size 1.27 1.27)))
-    )
-    (property "Value" "4.7kΩ"
-      (at 50 26.5 0)
-      (effects (font (size 1.27 1.27)))
-    )
-    (property "Footprint" "Resistor_SMD:R_0402_1005Metric"
-      (at 50 25 0)
-      (effects (font (size 1.27 1.27)) hide)
-    )
-    (instances
-      (project "uno_q_hub75_shield"
-        (path "/bc84562d-846a-4607-81a1-500b7991d137/3b4c5d6e-7f8a-9b0c-1d2e-3f4a5b6c7d8e"
-          (reference "R20") (unit 1)
-        )
-      )
-    )
-  )
-  (symbol (lib_id "Device:R")
-    (at 55 25 0)
-    (unit 1)
-    (in_bom yes) (on_board yes)
-    (property "Reference" "R21"
-      (at 55 23.5 0)
-      (effects (font (size 1.27 1.27)))
-    )
-    (property "Value" "4.7kΩ"
-      (at 55 26.5 0)
-      (effects (font (size 1.27 1.27)))
-    )
-    (property "Footprint" "Resistor_SMD:R_0402_1005Metric"
-      (at 55 25 0)
-      (effects (font (size 1.27 1.27)) hide)
-    )
-    (instances
-      (project "uno_q_hub75_shield"
-        (path "/bc84562d-846a-4607-81a1-500b7991d137/3b4c5d6e-7f8a-9b0c-1d2e-3f4a5b6c7d8e"
-          (reference "R21") (unit 1)
-        )
-      )
-    )
-  )
-  (symbol (lib_id "Device:R")
-    (at 60 30 0)
-    (unit 1)
-    (in_bom yes) (on_board yes)
-    (property "Reference" "JP1"
-      (at 60 28.5 0)
-      (effects (font (size 1.27 1.27)))
-    )
-    (property "Value" "0Ω"
-      (at 60 31.5 0)
-      (effects (font (size 1.27 1.27)))
-    )
-    (property "Footprint" "Resistor_SMD:R_0402_1005Metric"
-      (at 60 30 0)
-      (effects (font (size 1.27 1.27)) hide)
-    )
-    (instances
-      (project "uno_q_hub75_shield"
-        (path "/bc84562d-846a-4607-81a1-500b7991d137/3b4c5d6e-7f8a-9b0c-1d2e-3f4a5b6c7d8e"
-          (reference "JP1") (unit 1)
-        )
-      )
-    )
-  )
-  (hierarchical_label "+3V3"
-    (shape input)
-    (at 10 25 0)
-    (effects (font (size 1.27 1.27)) (justify left))
-  )
-  (hierarchical_label "+5V_BL"
-    (shape input)
-    (at 10 30 0)
-    (effects (font (size 1.27 1.27)) (justify left))
-  )
-  (hierarchical_label "LCD_CLK"
-    (shape input)
-    (at 10 35 0)
-    (effects (font (size 1.27 1.27)) (justify left))
-  )
-  (hierarchical_label "LCD_MOSI"
-    (shape input)
-    (at 10 40 0)
-    (effects (font (size 1.27 1.27)) (justify left))
-  )
-  (hierarchical_label "LCD_CS"
-    (shape input)
-    (at 10 45 0)
-    (effects (font (size 1.27 1.27)) (justify left))
-  )
-  (hierarchical_label "LCD_DC"
-    (shape input)
-    (at 10 50 0)
-    (effects (font (size 1.27 1.27)) (justify left))
-  )
-  (hierarchical_label "LCD_RST"
-    (shape input)
-    (at 10 55 0)
-    (effects (font (size 1.27 1.27)) (justify left))
-  )
-  (hierarchical_label "LCD_BL_PWM"
-    (shape input)
-    (at 10 60 0)
-    (effects (font (size 1.27 1.27)) (justify left))
-  )
-  (hierarchical_label "I2C_SDA"
-    (shape input)
-    (at 10 65 0)
-    (effects (font (size 1.27 1.27)) (justify left))
-  )
-  (hierarchical_label "I2C_SCL"
-    (shape input)
-    (at 10 70 0)
-    (effects (font (size 1.27 1.27)) (justify left))
-  )
-  (hierarchical_label "TOUCH_INT"
-    (shape input)
-    (at 10 75 0)
-    (effects (font (size 1.27 1.27)) (justify left))
-  )
+  (hierarchical_label "+3V3" (shape input) (at 10 25 0) (effects (font (size 1.27 1.27)) (justify right)) (uuid "hl9"))
   (sheet_instances
-    (path "/"
-      (page "1")
-    )
+    (path "/" (page "6"))
   )
 )
