File: KiCad/shield/sheets/display.kicad_sch (KiCad schematic)
At the start: 0 parts

Commit message: Populate shield schematics with actual components from BOM/DESIGN_SPEC
Power sheet: J4 barrel jack, C1/C2 bulk+bypass, U4 AMS1117-3.3,
  C3-C5 regulator caps, D1/D2 LEDs, R1/R2 current limiters

ESP32-S3 sheet: U1 ESP32-S3-WROOM-1-N16R8, R10/R11 pullups,
  C10/C11 bypass, J5 USB-C, R12/R13 CC resistors,
  All 20 GPIO hierarchical labels connected

HUB75 Driver: U2/U3 SN74HCT245PW level shifters, J1 HUB75 IDC,
  C16/C17 bypass caps, 0R DIR/OE ties to GND

Audio Codec: U5 ES8388, FB1 ferrite, C6-C9 supply caps,
  R3/R4 I2C pullups, C12-C15 DC blocking, J_OUT/J_MIC headers

Display: J6 Molex 503480-2200 22-pin FPC, R20/R21 GT911 pullups,
  C20/C21 bypass caps, JP1 SPI mode select

UNO Q Interface: J2 SPI header, J3 debug UART header

Connectivity: J8/J9 Qwiic, R5/R6 pullups, J10-J14 Grove connectors
Parts:
- added C20: 100nF, Capacitor_SMD:C_0402_1005Metric, symbol Device:C
- added C21: 10uF, Capacitor_SMD:C_0805_2012Metric, symbol Device:C
- added J6: 5in TFT+GT911, Connector_FFC-FPC:Molex_505068-2291_1x22-1MP_P0.50mm_Horizontal, symbol Connector:FPC-22
- added JP1: SPI_Mode, Jumper:SolderJumper-2_P1.3mm_Open_Pad1.0x1.5mm, symbol Device:SolderJumper_2_Open
- added R20, R21: 4.7k, Resistor_SMD:R_0402_1005Metric, symbol Device:R
