File: KiCad/shield/sheets/hub75_driver.kicad_sch (KiCad schematic)
At the start: 5 parts, among them J1 HUB75 Panel, U2 SN74HCT245, U3 SN74HCT245

Commit message: Use only standard KiCad libraries - remove HybotixParts dependency
Replaced all custom HybotixParts component references with standard KiCad libraries:
- BarrelJack_5V → Connector:Conn_01x02_Pin
- AMS1117-3.3 → Regulator_Linear:AMS1117-3.3
- ESP32-S3-WROOM-1-N16R8 → Module:ESP32-WROOM-32
- SN74HCT245PW → Logic_Inverter:SN74HCT245
- ES8388 → Audio:ES8388
- USB-C → Connector:USB_C_Receptacle_usb2.0
- FPC connectors → standard Connector parts
- All others mapped to nearest KiCad library equivalent

Removed embedded symbols section - all components now use standard KiCad built-in libraries.

All 16 schematics verified to parse correctly.
No external dependencies - ready to open in KiCad 10.0.2 on any machine.
Parts:
- J1: symbol HybotixParts:HUB75_2x8_IDC -> Connector:Conn_02x08_Odd_Even
- U2, U3: symbol HybotixParts:SN74HCT245PW -> Logic_Inverter:SN74HCT245
Changed lines of the file:
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@@
   (generator_version "10.0.0")
   (paper "A4")
-  (symbol (lib_id "HybotixParts:SN74HCT245PW")
+  (symbol (lib_id "Logic_Inverter:SN74HCT245")
     (at 30 25 0)
     (unit 1)
@@
     )
   )
-  (symbol (lib_id "HybotixParts:SN74HCT245PW")
+  (symbol (lib_id "Logic_Inverter:SN74HCT245")
     (at 30 45 0)
     (unit 1)
@@
     )
   )
-  (symbol (lib_id "HybotixParts:HUB75_2x8_IDC")
+  (symbol (lib_id "Connector:Conn_02x08_Odd_Even")
     (at 60 35 0)
     (unit 1)
