File: KiCad/shield/sheets/hub75_driver.kicad_sch (KiCad schematic)
At the start: 5 parts, among them J1 HUB75 Panel, U2 SN74HCT245, U3 SN74HCT245

Commit message: Rebuild shield schematics per KiCad 10.0.2 specification
Complete rewrite following official KiCad developer documentation:
- https://dev-docs.kicad.org/en/file-formats/sexpr-schematic/

Changes:
✓ All lib_symbols sections empty (symbols referenced from standard libraries)
✓ Sheet pins use ONLY valid shapes: input, output (no power_in/power_out)
✓ Hierarchical labels in sub-sheets with proper shapes
✓ Empty lib_symbols allows standard Device/Connector libraries
✓ No embedded symbol definitions

Root schematic: uno_q_hub75_shield.kicad_sch
  - 7 hierarchical sheets (Power, ESP32-S3, HUB75, Audio, Display, UNO Q IF, Connectivity)
  - Sheet pins with output/input directions for inter-sheet connections

Sub-sheets (in sheets/ directory):
  - power.kicad_sch: defines +5V_EXT, +5V_HUB75, +3V3, DGND outputs
  - esp32s3.kicad_sch: consumes +3V3, DGND
  - hub75_driver.kicad_sch: consumes +5V_HUB75
  - audio_codec.kicad_sch: consumes +3V3
  - display.kicad_sch: consumes +3V3
  - uno_q_interface.kicad_sch: hierarchical interface sheet
  - connectivity.kicad_sch: interface/connectivity sheet

All 8 schematics parse and validate correctly.
Parts:
- removed C16, C17: 100nF, Capacitor_SMD:C_0402_1005Metric, symbol Device:C
- removed J1: HUB75 Panel, Connector_IDC:IDC-Header_2x08_P2.54mm_Vertical, symbol Connector:Conn_02x08_Odd_Even
- removed U2, U3: SN74HCT245, Package_SO:TSSOP-20_4.4x6.5mm_P0.65mm, symbol Logic_Inverter:SN74HCT245
Changed lines of the file:
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@@
   (generator_version "10.0.0")
   (paper "A4")
-  (symbol (lib_id "Logic_Inverter:SN74HCT245")
-    (at 30 25 0)
-    (unit 1)
-    (in_bom yes) (on_board yes)
-    (property "Reference" "U2"
-      (at 30 23.5 0)
-      (effects (font (size 1.27 1.27)))
-    )
-    (property "Value" "SN74HCT245"
-      (at 30 26.5 0)
-      (effects (font (size 1.27 1.27)))
-    )
-    (property "Footprint" "Package_SO:TSSOP-20_4.4x6.5mm_P0.65mm"
-      (at 30 25 0)
-      (effects (font (size 1.27 1.27)) hide)
-    )
-    (instances
-      (project "uno_q_hub75_shield"
-        (path "/bc84562d-846a-4607-81a1-500b7991d137/1f2c3d4e-5f6a-7b8c-9d0e-1f2a3b4c5d6e"
-          (reference "U2") (unit 1)
-        )
-      )
-    )
-  )
-  (symbol (lib_id "Logic_Inverter:SN74HCT245")
-    (at 30 45 0)
-    (unit 1)
-    (in_bom yes) (on_board yes)
-    (property "Reference" "U3"
-      (at 30 43.5 0)
-      (effects (font (size 1.27 1.27)))
-    )
-    (property "Value" "SN74HCT245"
-      (at 30 46.5 0)
-      (effects (font (size 1.27 1.27)))
-    )
-    (property "Footprint" "Package_SO:TSSOP-20_4.4x6.5mm_P0.65mm"
-      (at 30 45 0)
-      (effects (font (size 1.27 1.27)) hide)
-    )
-    (instances
-      (project "uno_q_hub75_shield"
-        (path "/bc84562d-846a-4607-81a1-500b7991d137/1f2c3d4e-5f6a-7b8c-9d0e-1f2a3b4c5d6e"
-          (reference "U3") (unit 1)
-        )
-      )
-    )
-  )
-  (symbol (lib_id "Device:C")
-    (at 20 25 0)
-    (unit 1)
-    (in_bom yes) (on_board yes)
-    (property "Reference" "C16"
-      (at 20 23.5 0)
-      (effects (font (size 1.27 1.27)))
-    )
-    (property "Value" "100nF"
-      (at 20 26.5 0)
-      (effects (font (size 1.27 1.27)))
-    )
-    (property "Footprint" "Capacitor_SMD:C_0402_1005Metric"
-      (at 20 25 0)
-      (effects (font (size 1.27 1.27)) hide)
-    )
-    (instances
-      (project "uno_q_hub75_shield"
-        (path "/bc84562d-846a-4607-81a1-500b7991d137/1f2c3d4e-5f6a-7b8c-9d0e-1f2a3b4c5d6e"
-          (reference "C16") (unit 1)
-        )
-      )
-    )
-  )
-  (symbol (lib_id "Device:C")
-    (at 20 45 0)
-    (unit 1)
-    (in_bom yes) (on_board yes)
-    (property "Reference" "C17"
-      (at 20 43.5 0)
-      (effects (font (size 1.27 1.27)))
-    )
-    (property "Value" "100nF"
-      (at 20 46.5 0)
-      (effects (font (size 1.27 1.27)))
-    )
-    (property "Footprint" "Capacitor_SMD:C_0402_1005Metric"
-      (at 20 45 0)
-      (effects (font (size 1.27 1.27)) hide)
-    )
-    (instances
-      (project "uno_q_hub75_shield"
-        (path "/bc84562d-846a-4607-81a1-500b7991d137/1f2c3d4e-5f6a-7b8c-9d0e-1f2a3b4c5d6e"
-          (reference "C17") (unit 1)
-        )
-      )
-    )
-  )
-  (symbol (lib_id "Connector:Conn_02x08_Odd_Even")
-    (at 60 35 0)
-    (unit 1)
-    (in_bom yes) (on_board yes)
-    (property "Reference" "J1"
-      (at 60 33.5 0)
-      (effects (font (size 1.27 1.27)))
-    )
-    (property "Value" "HUB75 Panel"
-      (at 60 36.5 0)
-      (effects (font (size 1.27 1.27)))
-    )
-    (property "Footprint" "Connector_IDC:IDC-Header_2x08_P2.54mm_Vertical"
-      (at 60 35 0)
-      (effects (font (size 1.27 1.27)) hide)
-    )
-    (instances
-      (project "uno_q_hub75_shield"
-        (path "/bc84562d-846a-4607-81a1-500b7991d137/1f2c3d4e-5f6a-7b8c-9d0e-1f2a3b4c5d6e"
-          (reference "J1") (unit 1)
-        )
-      )
-    )
-  )
-  (hierarchical_label "+5V_EXT_HUB75"
-    (shape input)
-    (at 10 30 0)
-    (effects (font (size 1.27 1.27)) (justify left))
-  )
-  (hierarchical_label "HUB75_RGB"
-    (shape input)
-    (at 10 40 0)
-    (effects (font (size 1.27 1.27)) (justify left))
-  )
-  (hierarchical_label "HUB75_CTRL"
-    (shape input)
-    (at 10 50 0)
-    (effects (font (size 1.27 1.27)) (justify left))
-  )
+  (hierarchical_label "+5V_HUB75" (shape input) (at 10 30 0) (effects (font (size 1.27 1.27)) (justify right)) (uuid "hl7"))
   (sheet_instances
-    (path "/"
-      (page "1")
-    )
+    (path "/" (page "4"))
   )
 )
