File: KiCad/shield/sheets/hub75_driver.kicad_sch (KiCad schematic)
At the start: 0 parts

Commit message: Populate shield schematics with actual components from BOM/DESIGN_SPEC
Power sheet: J4 barrel jack, C1/C2 bulk+bypass, U4 AMS1117-3.3,
  C3-C5 regulator caps, D1/D2 LEDs, R1/R2 current limiters

ESP32-S3 sheet: U1 ESP32-S3-WROOM-1-N16R8, R10/R11 pullups,
  C10/C11 bypass, J5 USB-C, R12/R13 CC resistors,
  All 20 GPIO hierarchical labels connected

HUB75 Driver: U2/U3 SN74HCT245PW level shifters, J1 HUB75 IDC,
  C16/C17 bypass caps, 0R DIR/OE ties to GND

Audio Codec: U5 ES8388, FB1 ferrite, C6-C9 supply caps,
  R3/R4 I2C pullups, C12-C15 DC blocking, J_OUT/J_MIC headers

Display: J6 Molex 503480-2200 22-pin FPC, R20/R21 GT911 pullups,
  C20/C21 bypass caps, JP1 SPI mode select

UNO Q Interface: J2 SPI header, J3 debug UART header

Connectivity: J8/J9 Qwiic, R5/R6 pullups, J10-J14 Grove connectors
Parts:
- added C16, C17: 100nF, Capacitor_SMD:C_0402_1005Metric, symbol Device:C
- added J1: HUB75, Connector_IDC:IDC_Header_2x08_P2.54mm_Vertical, symbol Connector:IDC-Header_2x08_P2.54mm_Vertical
- added R_U2_DIR, R_U2_OE, R_U3_DIR, R_U3_OE: 0R, Resistor_SMD:R_0402_1005Metric, symbol Device:R
- added U2, U3: SN74HCT245PW, Package_SO:TSSOP-20_4.4x6.5mm_P0.65mm, symbol Device:74HCT245
Changed lines of the file:
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@@
 	(generator_version "8.0")
 	(paper "A4")
-	(hierarchical_label "+5V_HUB75"
-		(shape input)
-		(at 10 25 0)
-		(fields_autoplaced yes)
-		(effects
-			(font
-				(size 1.27 1.27)
-			)
-			(justify left)
-		)
-		(uuid "1f2c3d4e-5f6a-7b8c-9d0e-1f2a3b4c5d6e-hl00")
-	)
-	(hierarchical_label "HUB75_RGB"
-		(shape input)
-		(at 10 30 0)
-		(fields_autoplaced yes)
-		(effects
-			(font
-				(size 1.27 1.27)
-			)
-			(justify left)
-		)
-		(uuid "1f2c3d4e-5f6a-7b8c-9d0e-1f2a3b4c5d6e-hl01")
-	)
-	(hierarchical_label "HUB75_CTRL"
-		(shape input)
-		(at 10 35 0)
-		(fields_autoplaced yes)
-		(effects
-			(font
-				(size 1.27 1.27)
-			)
-			(justify left)
-		)
-		(uuid "1f2c3d4e-5f6a-7b8c-9d0e-1f2a3b4c5d6e-hl02")
-	)
+  (hierarchical_label "+5V_HUB75"
+    (shape input)
+    (at 10 20 0)
+    (fields_autoplaced yes)
+    (effects (font (size 1.27 1.27)) (justify left))
+    (uuid "hl-hub75-5v-in")
+  )
+  (hierarchical_label "DGND"
+    (shape input)
+    (at 10 25 0)
+    (fields_autoplaced yes)
+    (effects (font (size 1.27 1.27)) (justify left))
+    (uuid "hl-hub75-dgnd-in")
+  )
+  (hierarchical_label "HUB75_RGB"
+    (shape input)
+    (at 10 40 0)
+    (fields_autoplaced yes)
+    (effects (font (size 1.27 1.27)) (justify left))
+    (uuid "hl-hub75-rgb-in")
+  )
+  (hierarchical_label "HUB75_CTRL"
+    (shape input)
+    (at 10 45 0)
+    (fields_autoplaced yes)
+    (effects (font (size 1.27 1.27)) (justify left))
+    (uuid "hl-hub75-ctrl-in")
+  )
+  (symbol (lib_id "Device:74HCT245")
+    (at 50 60 0)
+    (unit 1)
+    (in_bom yes) (on_board yes)
+    (uuid "u2-uuid")
+    (property "Reference" "U2" (at 52 58 0) (effects (font (size 1.27 1.27))))
+    (property "Value" "SN74HCT245PW" (at 52 62 0) (effects (font (size 1.27 1.27))))
+    (property "Footprint" "Package_SO:TSSOP-20_4.4x6.5mm_P0.65mm" (at 50 60 0) (effects (font (size 1.27 1.27)) (hide yes)))
+    (instances (project "uno_q_hub75_shield" (path "/bc84562d-846a-4607-81a1-500b7991d137/{}" (reference "U2") (unit 1))))
+  )
+  (symbol (lib_id "Device:C")
+    (at 65 45 0)
+    (unit 1)
+    (in_bom yes) (on_board yes)
+    (uuid "c16-uuid")
+    (property "Reference" "C16" (at 67 43 0) (effects (font (size 1.27 1.27))))
+    (property "Value" "100nF" (at 67 47 0) (effects (font (size 1.27 1.27))))
+    (property "Footprint" "Capacitor_SMD:C_0402_1005Metric" (at 65 45 0) (effects (font (size 1.27 1.27)) (hide yes)))
+    (instances (project "uno_q_hub75_shield" (path "/bc84562d-846a-4607-81a1-500b7991d137/{}" (reference "C16") (unit 1))))
+  )
+  (symbol (lib_id "Device:74HCT245")
+    (at 50 110 0)
+    (unit 1)
+    (in_bom yes) (on_board yes)
+    (uuid "u3-uuid")
+    (property "Reference" "U3" (at 52 108 0) (effects (font (size 1.27 1.27))))
+    (property "Value" "SN74HCT245PW" (at 52 112 0) (effects (font (size 1.27 1.27))))
+    (property "Footprint" "Package_SO:TSSOP-20_4.4x6.5mm_P0.65mm" (at 50 110 0) (effects (font (size 1.27 1.27)) (hide yes)))
+    (instances (project "uno_q_hub75_shield" (path "/bc84562d-846a-4607-81a1-500b7991d137/{}" (reference "U3") (unit 1))))
+  )
+  (symbol (lib_id "Device:C")
+    (at 65 95 0)
+    (unit 1)
+    (in_bom yes) (on_board yes)
+    (uuid "c17-uuid")
+    (property "Reference" "C17" (at 67 93 0) (effects (font (size 1.27 1.27))))
+    (property "Value" "100nF" (at 67 97 0) (effects (font (size 1.27 1.27))))
+    (property "Footprint" "Capacitor_SMD:C_0402_1005Metric" (at 65 95 0) (effects (font (size 1.27 1.27)) (hide yes)))
+    (instances (project "uno_q_hub75_shield" (path "/bc84562d-846a-4607-81a1-500b7991d137/{}" (reference "C17") (unit 1))))
+  )
+  (symbol (lib_id "Connector:IDC-Header_2x08_P2.54mm_Vertical")
+    (at 100 80 0)
+    (unit 1)
+    (in_bom yes) (on_board yes)
+    (uuid "j1-uuid")
+    (property "Reference" "J1" (at 102 78 0) (effects (font (size 1.27 1.27))))
+    (property "Value" "HUB75" (at 102 82 0) (effects (font (size 1.27 1.27))))
+    (property "Footprint" "Connector_IDC:IDC_Header_2x08_P2.54mm_Vertical" (at 100 80 0) (effects (font (size 1.27 1.27)) (hide yes)))
+    (instances (project "uno_q_hub75_shield" (path "/bc84562d-846a-4607-81a1-500b7991d137/{}" (reference "J1") (unit 1))))
+  )
+  (symbol (lib_id "Device:R")
+    (at 35 55 90)
+    (unit 1)
+    (in_bom yes) (on_board yes)
+    (uuid "r-u2-dir")
+    (property "Reference" "R_U2_DIR" (at 37 53 0) (effects (font (size 1.27 1.27))))
+    (property "Value" "0R" (at 37 57 0) (effects (font (size 1.27 1.27))))
+    (property "Footprint" "Resistor_SMD:R_0402_1005Metric" (at 35 55 0) (effects (font (size 1.27 1.27)) (hide yes)))
+    (instances (project "uno_q_hub75_shield" (path "/bc84562d-846a-4607-81a1-500b7991d137/{}" (reference "R_U2_DIR") (unit 1))))
+  )
+  (symbol (lib_id "Device:R")
+    (at 35 65 90)
+    (unit 1)
+    (in_bom yes) (on_board yes)
+    (uuid "r-u2-oe")
+    (property "Reference" "R_U2_OE" (at 37 63 0) (effects (font (size 1.27 1.27))))
+    (property "Value" "0R" (at 37 67 0) (effects (font (size 1.27 1.27))))
+    (property "Footprint" "Resistor_SMD:R_0402_1005Metric" (at 35 65 0) (effects (font (size 1.27 1.27)) (hide yes)))
+    (instances (project "uno_q_hub75_shield" (path "/bc84562d-846a-4607-81a1-500b7991d137/{}" (reference "R_U2_OE") (unit 1))))
+  )
+  (symbol (lib_id "Device:R")
+    (at 35 105 90)
+    (unit 1)
+    (in_bom yes) (on_board yes)
+    (uuid "r-u3-dir")
+    (property "Reference" "R_U3_DIR" (at 37 103 0) (effects (font (size 1.27 1.27))))
+    (property "Value" "0R" (at 37 107 0) (effects (font (size 1.27 1.27))))
+    (property "Footprint" "Resistor_SMD:R_0402_1005Metric" (at 35 105 0) (effects (font (size 1.27 1.27)) (hide yes)))
+    (instances (project "uno_q_hub75_shield" (path "/bc84562d-846a-4607-81a1-500b7991d137/{}" (reference "R_U3_DIR") (unit 1))))
+  )
+  (symbol (lib_id "Device:R")
+    (at 35 115 90)
+    (unit 1)
+    (in_bom yes) (on_board yes)
+    (uuid "r-u3-oe")
+    (property "Reference" "R_U3_OE" (at 37 113 0) (effects (font (size 1.27 1.27))))
+    (property "Value" "0R" (at 37 117 0) (effects (font (size 1.27 1.27))))
+    (property "Footprint" "Resistor_SMD:R_0402_1005Metric" (at 35 115 0) (effects (font (size 1.27 1.27)) (hide yes)))
+    (instances (project "uno_q_hub75_shield" (path "/bc84562d-846a-4607-81a1-500b7991d137/{}" (reference "R_U3_OE") (unit 1))))
+  )
 	(sheet_instances
 		(path "/"
