File: KiCad/shield/sheets/esp32s3.kicad_sch (KiCad schematic)
At the start: 6 parts, among them J5 USB-C Debug, U1 ESP32-S3-WROOM-1-N16R8

Commit message: Rebuild shield schematics per KiCad 10.0.2 specification
Complete rewrite following official KiCad developer documentation:
- https://dev-docs.kicad.org/en/file-formats/sexpr-schematic/

Changes:
✓ All lib_symbols sections empty (symbols referenced from standard libraries)
✓ Sheet pins use ONLY valid shapes: input, output (no power_in/power_out)
✓ Hierarchical labels in sub-sheets with proper shapes
✓ Empty lib_symbols allows standard Device/Connector libraries
✓ No embedded symbol definitions

Root schematic: uno_q_hub75_shield.kicad_sch
  - 7 hierarchical sheets (Power, ESP32-S3, HUB75, Audio, Display, UNO Q IF, Connectivity)
  - Sheet pins with output/input directions for inter-sheet connections

Sub-sheets (in sheets/ directory):
  - power.kicad_sch: defines +5V_EXT, +5V_HUB75, +3V3, DGND outputs
  - esp32s3.kicad_sch: consumes +3V3, DGND
  - hub75_driver.kicad_sch: consumes +5V_HUB75
  - audio_codec.kicad_sch: consumes +3V3
  - display.kicad_sch: consumes +3V3
  - uno_q_interface.kicad_sch: hierarchical interface sheet
  - connectivity.kicad_sch: interface/connectivity sheet

All 8 schematics parse and validate correctly.
Parts:
- removed C10: 100nF, Capacitor_SMD:C_0402_1005Metric, symbol Device:C
- removed C11: 10µF, Capacitor_SMD:C_0805_2012Metric, symbol Device:C
- removed J5: USB-C Debug, Connector_USB:USB_C_Receptacle_GCT_USB4135-GF-A_Horizontal, symbol Connector:USB_C_Receptacle_usb2.0
- removed R12, R13: 5.1kΩ, Resistor_SMD:R_0402_1005Metric, symbol Device:R
- removed U1: ESP32-S3-WROOM-1-N16R8, Package_BGA:ESP32-S3-WROOM-1_18x25.5mm_P0.5mm, symbol Module:ESP32-WROOM-32
Changed lines of the file:
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@@
   (generator_version "10.0.0")
   (paper "A4")
-  (symbol (lib_id "Module:ESP32-WROOM-32")
-    (at 30 30 0)
-    (unit 1)
-    (in_bom yes) (on_board yes)
-    (property "Reference" "U1"
-      (at 30 28.5 0)
-      (effects (font (size 1.27 1.27)))
-    )
-    (property "Value" "ESP32-S3-WROOM-1-N16R8"
-      (at 30 31.5 0)
-      (effects (font (size 1.27 1.27)))
-    )
-    (property "Footprint" "Package_BGA:ESP32-S3-WROOM-1_18x25.5mm_P0.5mm"
-      (at 30 30 0)
-      (effects (font (size 1.27 1.27)) hide)
-    )
-    (instances
-      (project "uno_q_hub75_shield"
-        (path "/bc84562d-846a-4607-81a1-500b7991d137/02ac644c-33d8-477e-a8a6-71ca0780d582"
-          (reference "U1") (unit 1)
-        )
-      )
-    )
-  )
-  (symbol (lib_id "Device:C")
-    (at 20 30 0)
-    (unit 1)
-    (in_bom yes) (on_board yes)
-    (property "Reference" "C10"
-      (at 20 28.5 0)
-      (effects (font (size 1.27 1.27)))
-    )
-    (property "Value" "100nF"
-      (at 20 31.5 0)
-      (effects (font (size 1.27 1.27)))
-    )
-    (property "Footprint" "Capacitor_SMD:C_0402_1005Metric"
-      (at 20 30 0)
-      (effects (font (size 1.27 1.27)) hide)
-    )
-    (instances
-      (project "uno_q_hub75_shield"
-        (path "/bc84562d-846a-4607-81a1-500b7991d137/02ac644c-33d8-477e-a8a6-71ca0780d582"
-          (reference "C10") (unit 1)
-        )
-      )
-    )
-  )
-  (symbol (lib_id "Device:C")
-    (at 25 30 0)
-    (unit 1)
-    (in_bom yes) (on_board yes)
-    (property "Reference" "C11"
-      (at 25 28.5 0)
-      (effects (font (size 1.27 1.27)))
-    )
-    (property "Value" "10µF"
-      (at 25 31.5 0)
-      (effects (font (size 1.27 1.27)))
-    )
-    (property "Footprint" "Capacitor_SMD:C_0805_2012Metric"
-      (at 25 30 0)
-      (effects (font (size 1.27 1.27)) hide)
-    )
-    (instances
-      (project "uno_q_hub75_shield"
-        (path "/bc84562d-846a-4607-81a1-500b7991d137/02ac644c-33d8-477e-a8a6-71ca0780d582"
-          (reference "C11") (unit 1)
-        )
-      )
-    )
-  )
-  (symbol (lib_id "Connector:USB_C_Receptacle_usb2.0")
-    (at 60 30 0)
-    (unit 1)
-    (in_bom yes) (on_board yes)
-    (property "Reference" "J5"
-      (at 60 28.5 0)
-      (effects (font (size 1.27 1.27)))
-    )
-    (property "Value" "USB-C Debug"
-      (at 60 31.5 0)
-      (effects (font (size 1.27 1.27)))
-    )
-    (property "Footprint" "Connector_USB:USB_C_Receptacle_GCT_USB4135-GF-A_Horizontal"
-      (at 60 30 0)
-      (effects (font (size 1.27 1.27)) hide)
-    )
-    (instances
-      (project "uno_q_hub75_shield"
-        (path "/bc84562d-846a-4607-81a1-500b7991d137/02ac644c-33d8-477e-a8a6-71ca0780d582"
-          (reference "J5") (unit 1)
-        )
-      )
-    )
-  )
-  (symbol (lib_id "Device:R")
-    (at 65 25 0)
-    (unit 1)
-    (in_bom yes) (on_board yes)
-    (property "Reference" "R12"
-      (at 65 23.5 0)
-      (effects (font (size 1.27 1.27)))
-    )
-    (property "Value" "5.1kΩ"
-      (at 65 26.5 0)
-      (effects (font (size 1.27 1.27)))
-    )
-    (property "Footprint" "Resistor_SMD:R_0402_1005Metric"
-      (at 65 25 0)
-      (effects (font (size 1.27 1.27)) hide)
-    )
-    (instances
-      (project "uno_q_hub75_shield"
-        (path "/bc84562d-846a-4607-81a1-500b7991d137/02ac644c-33d8-477e-a8a6-71ca0780d582"
-          (reference "R12") (unit 1)
-        )
-      )
-    )
-  )
-  (symbol (lib_id "Device:R")
-    (at 65 35 0)
-    (unit 1)
-    (in_bom yes) (on_board yes)
-    (property "Reference" "R13"
-      (at 65 33.5 0)
-      (effects (font (size 1.27 1.27)))
-    )
-    (property "Value" "5.1kΩ"
-      (at 65 36.5 0)
-      (effects (font (size 1.27 1.27)))
-    )
-    (property "Footprint" "Resistor_SMD:R_0402_1005Metric"
-      (at 65 35 0)
-      (effects (font (size 1.27 1.27)) hide)
-    )
-    (instances
-      (project "uno_q_hub75_shield"
-        (path "/bc84562d-846a-4607-81a1-500b7991d137/02ac644c-33d8-477e-a8a6-71ca0780d582"
-          (reference "R13") (unit 1)
-        )
-      )
-    )
-  )
-  (hierarchical_label "+3V3"
-    (shape input)
-    (at 10 30 0)
-    (effects (font (size 1.27 1.27)) (justify left))
-  )
-  (hierarchical_label "DGND"
-    (shape input)
-    (at 10 35 0)
-    (effects (font (size 1.27 1.27)) (justify left))
-  )
-  (hierarchical_label "SPI_MOSI"
-    (shape output)
-    (at 50 15 0)
-    (effects (font (size 1.27 1.27)) (justify left))
-  )
-  (hierarchical_label "SPI_MISO"
-    (shape output)
-    (at 50 20 0)
-    (effects (font (size 1.27 1.27)) (justify left))
-  )
-  (hierarchical_label "SPI_SCK"
-    (shape output)
-    (at 50 25 0)
-    (effects (font (size 1.27 1.27)) (justify left))
-  )
-  (hierarchical_label "CS_S3_MCU"
-    (shape output)
-    (at 50 30 0)
-    (effects (font (size 1.27 1.27)) (justify left))
-  )
+  (hierarchical_label "+3V3" (shape input) (at 10 30 0) (effects (font (size 1.27 1.27)) (justify right)) (uuid "hl5"))
+  (hierarchical_label "DGND" (shape input) (at 10 35 0) (effects (font (size 1.27 1.27)) (justify right)) (uuid "hl6"))
   (sheet_instances
-    (path "/"
-      (page "1")
-    )
+    (path "/" (page "3"))
   )
 )
