File: KiCad/shield/uno_q_hub75_shield.kicad_sch (KiCad schematic)
At the start: 0 parts

Commit message: Fix: correct property names Sheetname/Sheetfile, add stroke/fill blocks
Based on real KiCad 8/10 schematics found on GitHub:
- Property names are Sheetname and Sheetfile (not Sheet name / Sheet file)
- Each sheet requires stroke and fill blocks
- fields_autoplaced yes required
- effects with justify left bottom/top for properties
Other:
- added sheet Audio Codec (sheets/audio_codec.kicad_sch)
- added sheet Connectivity (sheets/connectivity.kicad_sch)
- added sheet Display (sheets/display.kicad_sch)
- added sheet ESP32-S3 (sheets/esp32s3.kicad_sch)
- added sheet HUB75 Driver (sheets/hub75_driver.kicad_sch)
- added sheet Power (sheets/power.kicad_sch)
- added sheet UNO Q Interface (sheets/uno_q_interface.kicad_sch)
- company: (none) -> Hybrid RobotiX

Commit message: Add generator_version to schematic header
Other:
- removed sheet Audio Codec
- removed sheet Connectivity
- removed sheet Display
- removed sheet ESP32-S3
- removed sheet HUB75 Driver
- removed sheet Power
- removed sheet UNO Q Interface
- company: Hybrid RobotiX -> (none)
