File: KiCad/carrier/uno_q_super_carrier.kicad_sch (KiCad schematic)
At the start: 0 parts

Commit message: Rebuild all schematics with correct KiCad 10.0.2 format
Using exact format confirmed working with KiCad 10.0.2 on macOS.
All 16 schematics rebuilt:
- Shield root + 7 sub-sheets with hierarchical labels
- Carrier root + 7 sub-sheets with hierarchical labels

Format verified:
- version 20260101 (KiCad 10.0.2 SEXPR_SCHEMATIC_FILE_VERSION)
- generator_version 8.0
- Correct Sheetname/Sheetfile property names
- stroke/fill blocks on sheet definitions
- Proper hierarchical labels with effects blocks
Other:
- added sheet Power (sheets/power.kicad_sch)
- sheet Display Chain ports: added none; removed +3V3, +5V, DGND
- sheet ESP32-C6 Radio ports: added none; removed +3V3, DGND, S3_C6_RX, S3_C6_TX
- sheet Expansion ports: added none; removed +3V3, DGND, I2C_SCL, I2C_SDA
- sheet Level Shift ports: added none; removed +3V3, DGND, VIN_1V8_REF
- sheet RPi5 Interface ports: added none; removed +3V3, +5V, DGND
- sheet UNO Q Mounting ports: added none; removed +3V3, +5V, CS_S3_MPU, DGND, S3_C6_RX, S3_C6_TX
